File: pcb/pcb-wires-first.kicad_pcb (KiCad board)
At the start: 2 copper layers, 1 part, among them U1 SLG47115V

Commit message: Drafting.
Parts:
- added C2: 100nF, Capacitor_SMD:C_0603_1608Metric, F.Cu at (110.0, 112.5)
- added C3: 100nF, Capacitor_SMD:C_0603_1608Metric, F.Cu at (110.0, 106.0)
- added D1: ON, Diode_SMD:D_0603_1608Metric, F.Cu at (113.8, 106.5)
- added D2: FAULT, Diode_SMD:D_0603_1608Metric, F.Cu at (113.8, 110.0)
- added J3: Conn_01x04, Connector_PinHeader_2.54mm:PinHeader_1x04_P2.54mm_Vertical, B.Cu at (106.0, 120.0)
- added J4: Conn_01x06, Connector_PinHeader_2.54mm:PinHeader_1x06_P2.54mm_Vertical, B.Cu at (118.0, 100.9)
- added R1: 510, Resistor_SMD:R_0603_1608Metric, F.Cu at (113.7, 104.5)
- added R2: 510, Resistor_SMD:R_0603_1608Metric, F.Cu at (114.0, 108.5)
- added REF**: PinHeader_1x06_P2.54mm_Vertical, Connector_PinHeader_2.54mm:PinHeader_1x06_P2.54mm_Vertical, F.Cu at (100.0, 100.0)
- added REF**: PinHeader_1x02_P2.54mm_Vertical, Connector_PinHeader_2.54mm:PinHeader_1x02_P2.54mm_Vertical, F.Cu at (104.0, 95.5)
- added SW1: SW_Push, Button_Switch_SMD:SW_SPST_B3U-1000P, F.Cu at (106.0, 103.7)
- added SW2: SW_Push, Button_Switch_SMD:SW_SPST_B3U-1000P, F.Cu at (106.0, 109.3)
- moved U1 31.4 mm to (110.1, 109.1)
Connections:
- U1 pad 1: unconnected-(U1-V_{DD}-Pad1) -> VDD
- U1 pad 10: unconnected-(U1-HV_GPO1-Pad10) -> Net-(J3-Pin_3)
- U1 pad 11: unconnected-(U1-V_{DD2}-Pad11) -> VDD2
- U1 pad 13: unconnected-(U1-HV_GND-Pad13) -> HV_GND
- U1 pad 14: unconnected-(U1-GPIO1-Pad14) -> Net-(J4-Pin_2)
- U1 pad 15: unconnected-(U1-SCL-Pad15) -> Net-(J4-Pin_5)
- U1 pad 16: unconnected-(U1-SDA-Pad16) -> Net-(J4-Pin_4)
- U1 pad 17: unconnected-(U1-GPIO4-Pad17) -> Net-(J4-Pin_3)
- U1 pad 18: unconnected-(U1-GND-Pad18) -> GND
- U1 pad 19: unconnected-(U1-GPIO5-Pad19) -> /turn-on-hw
- U1 pad 2: unconnected-(U1-GPIO0-Pad2) -> /turn-off-sw
- U1 pad 20: unconnected-(U1-GPIO6-Pad20) -> /turn-on-sw
- U1 pad 3: unconnected-(U1-GPI-Pad3) -> /turn-off-hw
- U1 pad 4: unconnected-(U1-HV_GND-Pad4) -> HV_GND
- U1 pad 6: unconnected-(U1-V_{DD2}-Pad6) -> VDD2
- U1 pad 7: unconnected-(U1-HV_GPO0-Pad7) -> Net-(J3-Pin_2)
- U1 pad 8: unconnected-(U1-HV_GPO0-Pad8) -> Net-(J3-Pin_2)
- U1 pad 9: unconnected-(U1-HV_GPO1-Pad9) -> Net-(J3-Pin_3)
Other:
- board outline added: 24 x 28.5 mm

Commit message: Drafting the board.
Parts:
- removed J3: Conn_01x04, Connector_PinHeader_2.54mm:PinHeader_1x04_P2.54mm_Vertical
- removed J4: Conn_01x06, Connector_PinHeader_2.54mm:PinHeader_1x06_P2.54mm_Vertical
- removed REF**: PinHeader_1x06_P2.54mm_Vertical, Connector_PinHeader_2.54mm:PinHeader_1x06_P2.54mm_Vertical
- removed REF**: PinHeader_1x02_P2.54mm_Vertical, Connector_PinHeader_2.54mm:PinHeader_1x02_P2.54mm_Vertical
- added A1: Arduino_Nano_ESP32, Module:Arduino_Nano, F.Cu at (95.6, 124.5)
- added C10: 100nF, Capacitor_SMD:C_0603_1608Metric, F.Cu at (58.8, 109.5)
- added C11: 100nF, Capacitor_SMD:C_0603_1608Metric, F.Cu at (58.8, 107.5)
- added C12: 100nF, Capacitor_SMD:C_0603_1608Metric, F.Cu at (68.5, 103.3)
- added C13: 100nF, Capacitor_SMD:C_0603_1608Metric, F.Cu at (66.5, 103.3)
- added C14: 100nF, Capacitor_SMD:C_0603_1608Metric, F.Cu at (64.5, 103.3)
- added C15: 100nF, Capacitor_SMD:C_0603_1608Metric, F.Cu at (62.5, 103.3)
- added C16: 100nF, Capacitor_SMD:C_0603_1608Metric, F.Cu at (60.5, 105.0)
- added C4: 100nF, Capacitor_SMD:C_0603_1608Metric, F.Cu at (68.5, 112.8)
- added C5: 100nF, Capacitor_SMD:C_0603_1608Metric, F.Cu at (64.5, 112.8)
- added C6: 100nF, Capacitor_SMD:C_0603_1608Metric, F.Cu at (66.5, 112.8)
- added C7: 100nF, Capacitor_SMD:C_0603_1608Metric, F.Cu at (62.5, 112.8)
- added C8: 100nF, Capacitor_SMD:C_0603_1608Metric, F.Cu at (58.8, 113.5)
- added C9: 100nF, Capacitor_SMD:C_0603_1608Metric, F.Cu at (58.8, 111.5)
- added D3: ON, Diode_SMD:D_0603_1608Metric, F.Cu at (105.5, 108.5)
- added D4: ON, Diode_SMD:D_0603_1608Metric, F.Cu at (109.3, 119.1)
- added J10: Conn_01x02, Connector_Phoenix_MC:PhoenixContact_MCV_1,5_2-G-3.5_1x02_P3.50mm_Vertical, F.Cu at (123.0, 134.5)
- added J11: Conn_01x02, Connector_Phoenix_MC:PhoenixContact_MCV_1,5_2-G-3.5_1x02_P3.50mm_Vertical, F.Cu at (113.0, 134.5)
- added J2: Conn_01x02, Connector_Phoenix_MSTB:PhoenixContact_MSTBVA_2,5_2-G-5,08_1x02_P5.08mm_Vertical, F.Cu at (134.0, 95.6)
- added J5: Conn_01x04, Connector_Phoenix_MC:PhoenixContact_MCV_1,5_4-G-3.5_1x04_P3.50mm_Vertical, F.Cu at (49.0, 134.5)
- added J6: Conn_01x04, Connector_Phoenix_MC:PhoenixContact_MCV_1,5_4-G-3.5_1x04_P3.50mm_Vertical, F.Cu at (66.0, 134.5)
- added J7: Conn_01x04, Connector_Phoenix_MC:PhoenixContact_MCV_1,5_4-G-3.5_1x04_P3.50mm_Vertical, F.Cu at (83.0, 134.5)
- added J9: Conn_01x02, Connector_Phoenix_MC:PhoenixContact_MCV_1,5_2-G-3.5_1x02_P3.50mm_Vertical, F.Cu at (103.0, 134.5)
- added R3: 510, Resistor_SMD:R_0603_1608Metric, F.Cu at (110.2, 105.0)
- added R4: 510, Resistor_SMD:R_0603_1608Metric, F.Cu at (105.2, 117.8)
- added SW3: on-1, Button_Switch_SMD:SW_SPST_B3U-1000P, F.Cu at (54.8, 108.5)
- added SW4: off-1, Button_Switch_SMD:SW_SPST_B3U-1000P, F.Cu at (54.8, 112.0)
- added SW5: on-3, Button_Switch_SMD:SW_SPST_B3U-1000P, F.Cu at (67.0, 99.3)
- added SW6: off-3, Button_Switch_SMD:SW_SPST_B3U-1000P, F.Cu at (63.5, 99.3)
- added U2: SLG46826V, Package_DFN_QFN:Renesas_UQFN-20_2x3mm_P0.4mm_LayoutBorder4x6y, F.Cu at (64.0, 108.1)
- added U3: R-78C3.3-1.0, Converter_DCDC:Converter_DCDC_RECOM_R-78E-0.5_THT, F.Cu at (118.0, 90.9)
- SW1: value SW_Push -> off-2
- SW2: value SW_Push -> on-2
- moved SW2 43.2 mm to (63.5, 116.8), turned to -90 degrees
- moved SW1 41.1 mm to (67.0, 116.8), turned to -90 degrees
- moved R1 14.8 mm to (116.5, 119.0)
- moved D2 12.5 mm to (110.2, 122.0)
- moved C2 11.1 mm to (105.2, 122.5)
- moved D1 11.1 mm to (109.0, 116.5)
- moved R2 11.1 mm to (109.2, 118.5)
- moved U1 3.51 mm to (112.7, 111.5)
- moved C3 1.80 mm to (111.5, 107.0), turned to 180 degrees
Connections:
- C2 pad 1: HV_GND -> GND
- D2 pad 1: GND -> unconnected-(D2-K-Pad1)
- R1 pad 1: Net-(J4-Pin_3) -> Net-(A1-A2)
- R2 pad 1: Net-(J4-Pin_2) -> unconnected-(R2-Pad1)
- SW1 pad 1: GND -> /off-2a
- SW1 pad 2: /turn-off-sw -> GND
- SW2 pad 1: GND -> /on-2a
- SW2 pad 2: /turn-on-sw -> GND
- U1 pad 10: Net-(J3-Pin_3) -> unconnected-(U1-HV_GPO3-Pad10)
- U1 pad 13: HV_GND -> GND
- U1 pad 14: Net-(J4-Pin_2) -> Net-(A1-A1)
- U1 pad 15: Net-(J4-Pin_5) -> unconnected-(U1-SCL-Pad15)
- U1 pad 16: Net-(J4-Pin_4) -> unconnected-(U1-SDA-Pad16)
- U1 pad 17: Net-(J4-Pin_3) -> Net-(A1-A0)
- U1 pad 19: /turn-on-hw -> unconnected-(U1-GPIO5-Pad19)
- U1 pad 2: /turn-off-sw -> Net-(A1-A2)
- U1 pad 20: /turn-on-sw -> unconnected-(U1-GPIO6-Pad20)
- U1 pad 3: /turn-off-hw -> unconnected-(U1-GPI-Pad3)
- U1 pad 4: HV_GND -> GND
- U1 pad 7: Net-(J3-Pin_2) -> Net-(J11-Pin_2)
- U1 pad 8: Net-(J3-Pin_2) -> Net-(J10-Pin_2)
- U1 pad 9: Net-(J3-Pin_3) -> Net-(J9-Pin_2)
Routing:
- net /on-1a: track 0.00 -> 36.0 mm
- net /on-1b: track 0.00 -> 33.5 mm
- net /off-2b: track 0.00 -> 31.5 mm
- net /off-1a: track 0.00 -> 31.3 mm
- net /off-2a: track 0.00 -> 29.8 mm
- net /on-2a: track 0.00 -> 28.0 mm
- net /off-1b: track 0.00 -> 27.5 mm
- net /on-2b: track 0.00 -> 27.4 mm
- net /on-3a: track 0.00 -> 9.46 mm
- net /off-3a: track 0.00 -> 6.25 mm
- net /on-3b: track 0.00 -> 3.78 mm
- net /off-3b: track 0.00 -> 2.76 mm
- net VDD: track 0.00 -> 2.56 mm
Other:
- board size 24 x 28.5 mm -> 93.7 x 67 mm

Commit message: WIP.
Parts:
- added H1: MountingHole, MountingHole:MountingHole_3.2mm_M3, F.Cu at (49.5, 76.0)
- added H2: MountingHole, MountingHole:MountingHole_3.2mm_M3, F.Cu at (104.5, 85.9)
- added H3: MountingHole, MountingHole:MountingHole_3.2mm_M3, F.Cu at (104.5, 93.9)
- added H4: MountingHole, MountingHole:MountingHole_3.2mm_M3, F.Cu at (104.5, 101.8)
- J10, J11, J9: footprint Connector_Phoenix_MC:PhoenixContact_MCV_1,5_2-G-3.5_1x02_P3.50mm_Vertical -> Connector_JST:JST_VH_B2P-VH-FB-B_1x02_P3.96mm_Vertical
- J2: footprint Connector_Phoenix_MSTB:PhoenixContact_MSTBVA_2,5_2-G-5,08_1x02_P5.08mm_Vertical -> Connector_JST:JST_VH_B2P-VH-FB-B_1x02_P3.96mm_Vertical
- moved J10 3.23 mm to (125.5, 132.5)
- moved J11 2.55 mm to (114.6, 132.5)
- moved J9 2.07 mm to (103.5, 132.5)

Commit message: WIP.
Parts:
- added C1: 4.7μF/50V, Capacitor_SMD:C_1206_3216Metric, F.Cu at (124.3, 83.3)
- added C17: 10μF/50V, Capacitor_SMD:C_1206_3216Metric, F.Cu at (124.3, 86.7)
- added C18: 4.7μF/16V, Capacitor_SMD:C_0603_1608Metric, F.Cu at (136.0, 81.8)
- added D5: FAULT, Diode_SMD:D_0603_1608Metric, F.Cu at (129.2, 82.9)
- added L1: 10μF/4A, Inductor_SMD:L_Bourns_SRP7028A_7.3x6.6mm, F.Cu at (126.5, 77.6)
- added R5: 510, Resistor_SMD:R_0603_1608Metric, F.Cu at (129.2, 85.5)
- moved D3 3.24 mm to (104.3, 111.5)
- moved R3 3.01 mm to (110.0, 102.0)
- moved U1 1.00 mm to (112.7, 112.5)
Connections:
- net Net-(J10-Pin_2) renamed /output-2
- net Net-(J11-Pin_2) renamed /output-1
- net Net-(J9-Pin_2) renamed /output-3
- A1 pad 17: unconnected-(A1-3V3-Pad17) -> Net-(A1-3V3)
- A1 pad 29: Net-(A1-GND-Pad29) -> GND
- A1 pad 30: VDD -> unconnected-(A1-VIN-Pad30)
- A1 pad 4: Net-(A1-GND-Pad29) -> GND
- C16 pad 2: VDD -> 3V3
- C2 pad 1: GND -> HV-GND
- C2 pad 2: VDD2 -> HV-VDD
- C3 pad 2: VDD -> 3V3
- J10 pad 1: GND -> HV-GND
- J11 pad 1: GND -> HV-GND
- J2 pad 1: GND -> HV-GND
- J2 pad 2: VDD2 -> /hv-in-1
- J9 pad 1: GND -> HV-GND
- U1 pad 1: VDD -> 3V3
- U1 pad 11: VDD2 -> HV-VDD
- U1 pad 13: GND -> HV-GND
- U1 pad 19: unconnected-(U1-GPIO5-Pad19) -> Net-(U1-GPIO5)
- U1 pad 4: GND -> HV-GND
- U1 pad 6: VDD2 -> HV-VDD
- U2 pad 1: VDD -> 3V3
- U2 pad 14: unconnected-(U2-V_{DD2}-Pad14) -> 3V3
- U3 pad 1: VDD2 -> HV-VDD
- U3 pad 3: VDD -> 3V3
Routing:
- net VDD: track 2.56 -> 0.00 mm
- net 3V3: track 0.00 -> 2.56 mm

Commit message: Routing the board.
Parts:
- added D6: HV, Diode_SMD:D_0603_1608Metric, F.Cu at (161.5, 107.0)
- added R6: 6.7k, Resistor_SMD:R_0603_1608Metric, F.Cu at (158.0, 107.0)
- D1: value ON -> ON1
- D2: value FAULT -> ON2
- D3: value ON -> ON3
- D4: value ON -> FAULT
- D5: value FAULT -> 3V3
- R1, R2, R3, R4, R5: value 510 -> 2.2k
- moved H4 71.6 mm to (165.0, 140.0)
- moved H2 60.8 mm to (165.0, 80.0)
- moved H3 60.7 mm to (65.0, 140.0)
- moved SW6 58.8 mm to (113.0, 131.0)
- moved D3 57.3 mm to (161.5, 114.0), turned to 180 degrees
- moved D1 52.9 mm to (161.5, 110.0), turned to 180 degrees
- moved R4 52.8 mm to (158.0, 117.0)
- moved D4 52.3 mm to (161.5, 117.0), turned to 180 degrees
- moved D2 52.3 mm to (161.5, 112.0), turned to 180 degrees
- moved SW5 50.2 mm to (106.0, 131.0)
- moved J7 50.0 mm to (153.2, 138.2)
- moved R3 49.5 mm to (158.0, 114.0)
- moved R2 49.2 mm to (158.0, 112.0)
- moved R1 42.5 mm to (158.0, 110.0)
- moved D5 39.1 mm to (161.5, 105.0), turned to 180 degrees
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- renumbered C11 to C1, C12 to C10, C13 to C11, C14 to C12, C15 to C13, C3 to C14, C17 to C15, C2 to C16, C1 to C17, C10 to C2, C9 to C3, C8 to C4, C7 to C5, C5 to C6, C6 to C7, C4 to C8, C16 to C9, J5 to J1, J6 to J2, J7 to J3, J2 to J4, J11 to J5, J10 to J6, J9 to J7, SW3 to SW1, SW4 to SW2, SW2 to SW3, SW1 to SW4, U2 to U1, U1 to U2
Connections:
- net Net-(A1-A2) renamed switch-1
- A1 pad 19: Net-(A1-A0) -> switch-3
- A1 pad 20: Net-(A1-A1) -> switch-2
- A1 pad 22: unconnected-(A1-A3-Pad22) -> fault
- D2 pad 1: unconnected-(D2-K-Pad1) -> GND
- R2 pad 1: unconnected-(R2-Pad1) -> switch-2
- R3 pad 1: Net-(A1-A1) -> switch-3
- R4 pad 1: Net-(A1-A0) -> switch-3
- R5 pad 1: Net-(U1-GPIO5) -> 3V3
- U1 pad 15: Net-(A1-A1) -> switch-2
- U1 pad 16: Net-(A1-A0) -> switch-3
- U2 pad 14: Net-(A1-A1) -> switch-2
- U2 pad 17: Net-(A1-A0) -> switch-3
- U2 pad 19: Net-(U1-GPIO5) -> fault
Routing:
- net HV-GND: track 0.00 -> 86.0 mm
- net /off-3b: track 2.76 -> 75.4 mm, vias 0 -> 1
- net /on-3b: track 3.78 -> 69.9 mm, vias 0 -> 1
- net /off-1b: track 27.5 -> 76.1 mm, vias 0 -> 2
- net /on-2b: track 27.4 -> 74.6 mm, vias 0 -> 2
- net /on-1b: track 33.5 -> 78.1 mm, vias 0 -> 2
- net /off-3a: track 6.25 -> 50.0 mm
- net switch-3: track 0.00 -> 37.3 mm, vias 0 -> 1
- net switch-2: track 0.00 -> 36.0 mm, vias 0 -> 1
- net switch-1: track 0.00 -> 33.9 mm, vias 0 -> 1
- net /on-3a: track 9.46 -> 41.3 mm
- net /off-2b: track 31.5 -> 62.2 mm, vias 0 -> 1
- net /output-3: track 0.00 -> 28.2 mm
- net /output-1: track 0.00 -> 25.2 mm
- net /output-2: track 0.00 -> 23.9 mm
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Other:
- board size 93.7 x 67 mm -> 110 x 70 mm
