File: pcb/pcb-wires-first.kicad_sch (KiCad schematic)
At the start: 44 parts, among them J4 Conn_01x02, J5 OUT, J6 Conn_01x04, J8 I2C, SW7 set, SW8 reset, SW9 toggle, U2 SLG47115V, U3 R-78C3.3-1.0

Commit message: Debugging on a real board.
Parts:
- SW7: value set -> reset
- SW8: value reset -> set
Other:
- moved on the sheet: C18
Changed lines of the file:
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@@
 	)
 	(junction
+		(at 133.35 248.92)
+		(diameter 0)
+		(color 0 0 0 0)
+	)
+	(junction
 		(at 99.06 217.17)
 		(diameter 0)
@@
 	)
 	(junction
-		(at 133.35 248.92)
-		(diameter 0)
-		(color 0 0 0 0)
-	)
-	(junction
 		(at 292.1 86.36)
 		(diameter 0)
@@
 	(wire
 		(pts
-			(xy 133.35 226.06) (xy 133.35 248.92)
+			(xy 133.35 237.49) (xy 133.35 248.92)
 		)
 		(stroke
@@
 	(wire
 		(pts
-			(xy 133.35 217.17) (xy 133.35 218.44)
+			(xy 133.35 217.17) (xy 133.35 229.87)
 		)
 		(stroke
@@
 			)
 		)
-		(property "Value" "reset"
+		(property "Value" "set"
 			(at 287.02 91.186 0)
 			(show_name no)
@@
 	(symbol
 		(lib_id "Device:C")
-		(at 133.35 222.25 0)
+		(at 133.35 233.68 0)
 		(unit 1)
 		(body_style 1)
@@
 		(dnp no)
 		(property "Reference" "C18"
-			(at 132.08 227.33 90)
+			(at 132.08 238.76 90)
 			(show_name no)
 			(do_not_autoplace no)
@@
 		)
 		(property "Value" "4.7μF/16V"
-			(at 136.398 227.584 90)
+			(at 136.398 239.014 90)
 			(show_name no)
 			(do_not_autoplace no)
@@
 		)
 		(property "Footprint" "Capacitor_SMD:C_0603_1608Metric"
-			(at 134.3152 226.06 0)
+			(at 134.3152 237.49 0)
 			(hide yes)
 			(show_name no)
@@
 		)
 		(property "Datasheet" ""
-			(at 133.35 222.25 0)
+			(at 133.35 233.68 0)
 			(hide yes)
 			(show_name no)
@@
 		)
 		(property "Description" "Unpolarized capacitor"
-			(at 133.35 222.25 0)
+			(at 133.35 233.68 0)
 			(hide yes)
 			(show_name no)
@@
 			)
 		)
-		(property "Value" "set"
+		(property "Value" "reset"
 			(at 274.32 92.71 0)
 			(show_name no)
