File: pcb/switcher/switcher.kicad_pcb (KiCad board)
At the start: 2 copper layers, 37.4 x 47.4 mm, 36 parts, among them J4 Conn_01x02, J5 OUT, J6 Conn_01x04, J8 I2C, J9 I2C, SW7 reset, SW8 set, SW9 toggle, U2 SLG47115V

Commit message: Updating libraries mostly.
Parts:
- J6: value Conn_01x04 -> Input
- U2: footprint Package_DFN_QFN:Renesas_UQFN-20_2x3mm_P0.4mm_LayoutBorder4x6y -> Package_DFN_QFN:Renesas_UQFN-20_2x3mm_P0.4mm_SLG47115V
Changed lines of the file:
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@@
 		)
 	)
-	(footprint "Package_DFN_QFN:Renesas_UQFN-20_2x3mm_P0.4mm_LayoutBorder4x6y"
+	(footprint "Package_DFN_QFN:Renesas_UQFN-20_2x3mm_P0.4mm_SLG47115V"
 		(layer "F.Cu")
 		(at 94.875 115.4)
-		(descr "Renesas  UQFN, 20 Pin (Renesas STQFN-20L, https://www.renesas.com/en/document/dst/slg465808283-datasheet#page=200)")
-		(tags "Renesas UQFN NoLead")
+		(descr "Renesas  UQFN, 20 Pin, specific to SLG47115V")
+		(tags "Renesas UQFN NoLead SLG47115V")
 		(property "Reference" "U2"
-			(at 0.075 3.15 0)
+			(at 0 -2.8 0)
 			(layer "F.SilkS")
 			(effects
@@
 			)
 		)
+		(clearance 0.18)
 		(attr smd)
 		(duplicate_pad_numbers_are_jumpers no)
@@
 		(pad "1" smd roundrect
 			(at -1.025 -1)
-			(size 0.65 0.2)
+			(size 0.65 0.21)
 			(layers "F.Cu" "F.Mask" "F.Paste")
 			(roundrect_rratio 0.25)
@@
 		(pad "2" smd roundrect
 			(at -1.025 -0.6)
-			(size 0.65 0.2)
+			(size 0.65 0.21)
 			(layers "F.Cu" "F.Mask" "F.Paste")
 			(roundrect_rratio 0.25)
@@
 		(pad "3" smd roundrect
 			(at -1.025 -0.2)
-			(size 0.65 0.2)
+			(size 0.65 0.21)
 			(layers "F.Cu" "F.Mask" "F.Paste")
 			(roundrect_rratio 0.25)
@@
 		(pad "4" smd roundrect
 			(at -1.025 0.2)
-			(size 0.65 0.2)
+			(size 0.65 0.21)
 			(layers "F.Cu" "F.Mask" "F.Paste")
 			(roundrect_rratio 0.25)
@@
 			(pintype "power_in")
 		)
+		(pad "4" smd roundrect
+			(at -0.3 0.125)
+			(size 0.4 0.48)
+			(layers "F.Cu" "F.Mask" "F.Paste")
+			(roundrect_rratio 0.1204819277)
+			(net "HV-GND")
+			(pinfunction "HV_GND_4")
+			(pintype "power_in")
+		)
 		(pad "5" smd roundrect
 			(at -1.025 0.6)
-			(size 0.65 0.2)
+			(size 0.65 0.21)
 			(layers "F.Cu" "F.Mask" "F.Paste")
 			(roundrect_rratio 0.25)
@@
 		(pad "6" smd roundrect
 			(at -1.025 1)
-			(size 0.65 0.2)
+			(size 0.65 0.21)
 			(layers "F.Cu" "F.Mask" "F.Paste")
 			(roundrect_rratio 0.25)
@@
 		(pad "7" smd roundrect
 			(at -0.6 1.5625)
-			(size 0.2 0.575)
+			(size 0.21 0.575)
 			(layers "F.Cu" "F.Mask" "F.Paste")
 			(roundrect_rratio 0.25)
@@
 		)
 		(pad "8" smd roundrect
-			(at -0.2 1.525)
-			(size 0.2 0.65)
+			(at -0.2 1.38)
+			(size 0.21 0.94)
 			(layers "F.Cu" "F.Mask" "F.Paste")
 			(roundrect_rratio 0.25)
@@
 		)
 		(pad "9" smd roundrect
-			(at 0.2 1.525)
-			(size 0.2 0.65)
+			(at 0.2 1.38)
+			(size 0.21 0.94)
 			(layers "F.Cu" "F.Mask" "F.Paste")
 			(roundrect_rratio 0.25)
@@
 		(pad "10" smd roundrect
 			(at 0.6 1.5625)
-			(size 0.2 0.575)
+			(size 0.21 0.575)
 			(layers "F.Cu" "F.Mask" "F.Paste")
 			(roundrect_rratio 0.25)
@@
 		(pad "11" smd roundrect
 			(at 1.025 1)
-			(size 0.65 0.2)
+			(size 0.65 0.21)
 			(layers "F.Cu" "F.Mask" "F.Paste")
 			(roundrect_rratio 0.25)
@@
 		(pad "12" smd roundrect
 			(at 1.025 0.6)
-			(size 0.65 0.2)
+			(size 0.65 0.21)
 			(layers "F.Cu" "F.Mask" "F.Paste")
 			(roundrect_rratio 0.25)
@@
 		)
 		(pad "13" smd roundrect
+			(at 0.3 0.125)
+			(size 0.4 0.48)
+			(layers "F.Cu" "F.Mask" "F.Paste")
+			(roundrect_rratio 0.1204819277)
+			(net "HV-GND")
+			(pinfunction "HV_GND_13")
+			(pintype "power_in")
+		)
+		(pad "13" smd roundrect
 			(at 1.025 0.2)
-			(size 0.65 0.2)
+			(size 0.65 0.21)
 			(layers "F.Cu" "F.Mask" "F.Paste")
 			(roundrect_rratio 0.25)
@@
 		(pad "14" smd roundrect
 			(at 1.025 -0.2)
-			(size 0.65 0.2)
+			(size 0.65 0.21)
 			(layers "F.Cu" "F.Mask" "F.Paste")
 			(roundrect_rratio 0.25)
@@
 		(pad "15" smd roundrect
 			(at 1.025 -0.6)
-			(size 0.65 0.2)
+			(size 0.65 0.21)
 			(layers "F.Cu" "F.Mask" "F.Paste")
 			(roundrect_rratio 0.25)
@@
 		(pad "16" smd roundrect
 			(at 1.025 -1)
-			(size 0.65 0.2)
+			(size 0.65 0.21)
 			(layers "F.Cu" "F.Mask" "F.Paste")
 			(roundrect_rratio 0.25)
@@
 		(pad "17" smd roundrect
 			(at 0.6 -1.5625)
-			(size 0.2 0.575)
+			(size 0.21 0.575)
 			(layers "F.Cu" "F.Mask" "F.Paste")
 			(roundrect_rratio 0.25)
@@
 		)
 		(pad "18" smd roundrect
+			(at -0.3 -0.615)
+			(size 0.4 0.48)
+			(layers "F.Cu" "F.Mask" "F.Paste")
+			(roundrect_rratio 0.1204819277)
+			(net "GND")
+			(pinfunction "GND_18")
+			(pintype "power_in")
+		)
+		(pad "18" smd roundrect
 			(at 0.2 -1.525)
-			(size 0.2 0.65)
+			(size 0.21 0.65)
 			(layers "F.Cu" "F.Mask" "F.Paste")
 			(roundrect_rratio 0.25)
@@
 			(pintype "power_in")
 		)
+		(pad "18" smd roundrect
+			(at 0.3 -0.615)
+			(size 0.4 0.48)
+			(layers "F.Cu" "F.Mask" "F.Paste")
+			(roundrect_rratio 0.1204819277)
+			(net "GND")
+			(pinfunction "GND_18")
+			(pintype "power_in")
+		)
 		(pad "19" smd roundrect
 			(at -0.2 -1.475)
-			(size 0.2 0.75)
+			(size 0.21 0.75)
 			(layers "F.Cu" "F.Mask" "F.Paste")
 			(roundrect_rratio 0.25)
@@
 		(pad "20" smd roundrect
 			(at -0.6 -1.5625)
-			(size 0.2 0.575)
+			(size 0.21 0.575)
 			(layers "F.Cu" "F.Mask" "F.Paste")
 			(roundrect_rratio 0.25)
@@
 		)
 		(embedded_fonts no)
-		(model "${KICAD10_3DMODEL_DIR}/Package_DFN_QFN.3dshapes/Renesas_UQFN-20_2x3mm_P0.4mm_LayoutBorder4x6y.step"
+		(model "${KICAD10_3DMODEL_DIR}/Package_DFN_QFN.3dshapes/Renesas_UQFN-20_2x3mm_P0.4mm_SLG47115V.step"
 			(offset
 				(xyz 0 0 0)
@@
 			)
 			(rotate
-				(xyz 0 0 0)
+				(xyz -0 -0 -0)
 			)
 		)
@@
 			)
 		)
-		(property "Value" "Conn_01x04"
+		(property "Value" "Input"
 			(at 5.25 4.2 0)
 			(layer "F.Fab")
@@
 	(gr_poly
 		(pts
-			(xy 94.45 115) (xy 95.3 115) (xy 95.3 114.55) (xy 94.45 114.55)
-		)
-		(stroke
-			(width 0)
-			(type solid)
-		)
-		(fill yes)
-		(layer "F.Cu")
-		(net "GND")
-	)
-	(gr_poly
-		(pts
-			(xy 94.45 115.725) (xy 95.3 115.725) (xy 95.3 115.275) (xy 94.45 115.275)
-		)
-		(stroke
-			(width 0)
-			(type solid)
-		)
-		(fill yes)
-		(layer "F.Cu")
-		(net "HV-GND")
-	)
-	(gr_poly
-		(pts
 			(xy 94.975 114.1) (xy 94.975 114.625) (xy 95.175 114.625) (xy 95.175 114.1)
 		)
@@
 	)
 	(segment
-		(start 99.025 108.2875)
-		(end 98.2875 107.55)
-		(width 0.2)
-		(layer "F.Cu")
-		(net "Net-(D4-A)")
-	)
-	(segment
-		(start 99 111.175)
-		(end 99.025 111.15)
-		(width 0.2)
-		(layer "F.Cu")
-		(net "Net-(D4-A)")
-	)
-	(segment
-		(start 99.025 111.15)
-		(end 99.025 108.2875)
-		(width 0.2)
-		(layer "F.Cu")
-		(net "Net-(D4-A)")
-	)
-	(segment
-		(start 97.8 115.2)
-		(end 99 114)
-		(width 0.2)
-		(layer "F.Cu")
-		(net "Net-(U2-GPIO1)")
-	)
-	(segment
-		(start 99 114)
-		(end 99 112.825)
-		(width 0.2)
-		(layer "F.Cu")
-		(net "Net-(U2-GPIO1)")
-	)
-	(segment
-		(start 95.9 115.2)
-		(end 97.8 115.2)
-		(width 0.2)
-		(layer "F.Cu")
-		(net "Net-(U2-GPIO1)")
-	)
-	(segment
 		(start 95.9 114.4)
 		(end 96.90294 114.4)
@@
 	)
 	(segment
-		(start 89.75 105.65)
-		(end 89.75 112.95)
-		(width 2)
-		(layer "F.Cu")
-		(net "HV-VDD")
-	)
-	(segment
-		(start 93 105.65)
-		(end 100.75 105.65)
-		(width 2)
-		(layer "F.Cu")
-		(net "HV-VDD")
-	)
-	(segment
-		(start 89.75 105.65)
-		(end 93 105.65)
-		(width 2)
-		(layer "F.Cu")
-		(net "HV-VDD")
-	)
-	(segment
-		(start 93.04 105.61)
-		(end 93 105.65)
-		(width 2)
-		(layer "F.Cu")
-		(net "HV-VDD")
-	)
-	(segment
-		(start 100.75 117.55)
-		(end 99.75 118.55)
-		(width 2)
-		(layer "F.Cu")
-		(net "HV-VDD")
-	)
-	(segment
-		(start 93.04 102.05)
-		(end 93.04 105.61)
-		(width 2)
-		(layer "F.Cu")
-		(net "HV-VDD")
-	)
-	(segment
-		(start 100.75 105.65)
-		(end 100.75 117.55)
-		(width 2)
-		(layer "F.Cu")
-		(net "HV-VDD")
-	)
-	(segment
 		(start 92.55 113.1)
 		(end 92.55 112.35)
@@
 	)
 	(segment
+		(start 99.025 108.2875)
+		(end 98.2875 107.55)
+		(width 0.2)
+		(layer "F.Cu")
+		(net "Net-(D4-A)")
+	)
+	(segment
+		(start 99 111.175)
+		(end 99.025 111.15)
+		(width 0.2)
+		(layer "F.Cu")
+		(net "Net-(D4-A)")
+	)
+	(segment
+		(start 99.025 111.15)
+		(end 99.025 108.2875)
+		(width 0.2)
+		(layer "F.Cu")
+		(net "Net-(D4-A)")
+	)
+	(segment
+		(start 97.8 115.2)
+		(end 99 114)
+		(width 0.2)
+		(layer "F.Cu")
+		(net "Net-(U2-GPIO1)")
+	)
+	(segment
+		(start 99 114)
+		(end 99 112.825)
+		(width 0.2)
+		(layer "F.Cu")
+		(net "Net-(U2-GPIO1)")
+	)
+	(segment
+		(start 95.9 115.2)
+		(end 97.8 115.2)
+		(width 0.2)
+		(layer "F.Cu")
+		(net "Net-(U2-GPIO1)")
+	)
+	(segment
 		(start 93.5 129.8)
 		(end 93.4 129.7)
@@
 	)
 	(segment
+		(start 89.75 105.65)
+		(end 89.75 112.95)
+		(width 2)
+		(layer "F.Cu")
+		(net "HV-VDD")
+	)
+	(segment
+		(start 93 105.65)
+		(end 100.75 105.65)
+		(width 2)
+		(layer "F.Cu")
+		(net "HV-VDD")
+	)
+	(segment
+		(start 89.75 105.65)
+		(end 93 105.65)
+		(width 2)
+		(layer "F.Cu")
+		(net "HV-VDD")
+	)
+	(segment
+		(start 93.04 105.61)
+		(end 93 105.65)
+		(width 2)
+		(layer "F.Cu")
+		(net "HV-VDD")
+	)
+	(segment
+		(start 100.75 117.55)
+		(end 99.75 118.55)
+		(width 2)
+		(layer "F.Cu")
+		(net "HV-VDD")
+	)
+	(segment
+		(start 93.04 102.05)
+		(end 93.04 105.61)
+		(width 2)
+		(layer "F.Cu")
+		(net "HV-VDD")
+	)
+	(segment
+		(start 100.75 105.65)
+		(end 100.75 117.55)
+		(width 2)
+		(layer "F.Cu")
+		(net "HV-VDD")
+	)
+	(segment
