File: pcb/switcher/switcher.kicad_pcb (KiCad board)
At the start: 2 copper layers, 37.4 x 47.4 mm, 40 parts, among them J1 Input, J2 OUT, J3 Conn_01x02, J4 I2C, J5 I2C, SW1 toggle, SW2 reset, SW3 set, U1 SLG47115V

Commit message: Switcher: Adding TVS diodes.
Parts:
- added U2: TPD4E02B04DQA, Package_SON:USON-10_2.5x1.0mm_P0.5mm, F.Cu at (95.7, 134.4)
- RN1: value R_Pack04 -> 100
- moved RN1 9.73 mm to (95.8, 131.9)
- moved SW1 0.10 mm to (100.5, 127.8)
- moved SW2 0.10 mm to (97.0, 127.8)
- moved SW3 0.10 mm to (93.5, 127.8)
- renumbered JP1 to PU1, JP2 to PU2
Routing:
- net Net-(RN1-R4.2): track 41.6 -> 31.1 mm
- net Net-(RN1-R3.2): track 35.8 -> 25.5 mm
- net Net-(J1-Pin_4): track 17.9 -> 9.85 mm
- net Net-(J1-Pin_3): track 15.1 -> 7.72 mm
- net Net-(RN1-R2.2): track 29.5 -> 22.9 mm
- net Net-(J1-Pin_2): track 12.2 -> 8.18 mm
- net GND: track 2.68 -> 4.92 mm, vias 8 -> 17
