File: pcb/switcher/switcher.kicad_sch (KiCad schematic)
At the start: 36 parts, among them J4 Conn_01x02, J5 OUT, J6 Input, J8 I2C, J9 I2C, SW7 reset, SW8 set, SW9 toggle, U2 SLG47115V

Commit message: Updating libraries mostly.
Parts:
- U2: footprint Package_DFN_QFN:Renesas_UQFN-20_2x3mm_P0.4mm_LayoutBorder4x6y -> Package_DFN_QFN:Renesas_UQFN-20_2x3mm_P0.4mm_SLG47115V
Changed lines of the file:
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@@
 			)
 		)
-		(property "Footprint" "Package_DFN_QFN:Renesas_UQFN-20_2x3mm_P0.4mm_LayoutBorder4x6y"
+		(property "Footprint" "Package_DFN_QFN:Renesas_UQFN-20_2x3mm_P0.4mm_SLG47115V"
 			(at 125.476 168.91 0)
 			(hide yes)

Commit message: Preparing switcher for fabrication.
Parts:
- renumbered C20 to C1, C19 to C2, C22 to C3, C14 to C4, C16 to C5, C18 to C6, D4 to D1, D3 to D2, D2 to D3, D6 to D4, J6 to J1, J5 to J2, J4 to J3, J8 to J4, J9 to J5, NT4 to NT1, NT5 to NT2, NT2 to NT3, NT3 to NT4, R4 to R1, R3 to R2, R2 to R3, R6 to R4, R7 to R6, R8 to R7, SW9 to SW1, SW7 to SW2, SW8 to SW3, U2 to U1

Commit message: Adding issues after live testing and soldering.
Connections:
- net HV-GND: now also U1.12 (SENSE2), U1.5 (SENSE1)
- no-connect marks 3 -> 1
Other:
- note added: "ISSUES TO FIX IN ${VERSION} 1. SENSE should be tied to HV_GND - DONE 2. Thermal vias should be capped if possible 3. Control inputs aren't very protected 4. I2C pull upps shopuld be removed, or at least add solderable bridges"
Changed lines of the file:
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@@
 	(generator_version "10.0")
 	(paper "A3")
+	(title_block
+		(rev "${VERSION}")
+	)
 	(text "Switcher"
 		(exclude_from_sim no)
@@
 		)
 	)
+	(text "ISSUES TO FIX IN ${VERSION}\n\n1. SENSE should be tied to HV_GND - DONE\n2. Thermal vias should be capped if possible\n3. Control inputs aren't very protected\n4. I2C pull upps shopuld be removed, or at least add solderable bridges"
+		(exclude_from_sim no)
+		(at 368.808 25.908 0)
+		(effects
+			(font
+				(size 1.27 1.27)
+			)
+		)
+	)
 	(junction
 		(at 130.81 110.49)
@@
 	)
 	(junction
+		(at 106.68 146.05)
+		(diameter 0)
+		(color 0 0 0 0)
+	)
+	(junction
 		(at 130.81 156.21)
 		(diameter 0)
@@
 		(diameter 0)
 		(color 0 0 0 0)
-	)
-	(no_connect
-		(at 107.95 143.51)
 	)
 	(no_connect
 		(at 107.95 120.65)
 	)
-	(no_connect
-		(at 107.95 146.05)
-	)
 	(wire
 		(pts
@@
 	(wire
 		(pts
+			(xy 106.68 168.91) (xy 130.81 168.91)
+		)
+		(stroke
+			(width 0)
+			(type default)
+		)
+	)
+	(wire
+		(pts
 			(xy 86.36 137.16) (xy 88.9 137.16)
 		)
@@
 	(wire
 		(pts
+			(xy 106.68 143.51) (xy 106.68 146.05)
+		)
+		(stroke
+			(width 0)
+			(type default)
+		)
+	)
+	(wire
+		(pts
 			(xy 130.81 102.87) (xy 130.81 110.49)
 		)
@@
 	(wire
 		(pts
+			(xy 106.68 146.05) (xy 107.95 146.05)
+		)
+		(stroke
+			(width 0)
+			(type default)
+		)
+	)
+	(wire
+		(pts
 			(xy 86.36 149.86) (xy 88.9 149.86)
 		)
@@
 	(wire
 		(pts
+			(xy 106.68 146.05) (xy 106.68 168.91)
+		)
+		(stroke
+			(width 0)
+			(type default)
+		)
+	)
+	(wire
+		(pts
 			(xy 130.81 168.91) (xy 154.94 168.91)
 		)
@@
 		)
 		(stroke
+			(width 0)
+			(type default)
+		)
+	)
+	(wire
+		(pts
+			(xy 107.95 143.51) (xy 106.68 143.51)
+		)
+		(stroke
