File: pcb/gateway/gateway2/gateway2.kicad_pcb (KiCad board)
At the start: 2 copper layers, 45 parts, among them J1 Conn_01x07, J10 Conn_ARM_JTAG_SWD_10, J2 Conn_01x07, J3 Conn_01x07, J4 Conn_01x07, J5 Conn_01x07, J6 Conn_01x07, J7 Conn_01x07, J8 Conn_01x07, J9 RJ45_Kycon_G7LX-A88S7-BP-GY, U1 RP2354B, U2 W6300-Q

Commit message: Continuing draft. Adding sample projects, datasheets.
Parts:
- added C26: 100n, Capacitor_SMD:C_0603_1608Metric, F.Cu at (153.4, 101.4)
- added R13: 5k6, Resistor_SMD:R_0603_1608Metric, F.Cu at (153.4, 103.9)
- added R14: 10k, Resistor_SMD:R_0603_1608Metric, F.Cu at (153.4, 106.4)
- added R15: 100k, Resistor_SMD:R_0603_1608Metric, F.Cu at (153.4, 108.9)
- added R16: 27, Resistor_SMD:R_0603_1608Metric, F.Cu at (153.4, 111.4)
- added R17: R, Resistor_SMD:R_0603_1608Metric, F.Cu at (153.4, 113.9)
- added R18: 100, Resistor_SMD:R_0603_1608Metric, F.Cu at (157.4, 101.4)
- added R19: 100, Resistor_SMD:R_0603_1608Metric, F.Cu at (157.4, 103.9)
- added R20: 1k, Resistor_SMD:R_0603_1608Metric, F.Cu at (157.4, 106.4)
- added R21: 1k, Resistor_SMD:R_0603_1608Metric, F.Cu at (157.4, 108.9)
- added R22: 10k, Resistor_SMD:R_0603_1608Metric, F.Cu at (157.4, 111.4)
Connections:
- net Net-(U1-GPIO15) renamed ETH_INT
- net Net-(U1-GPIO22) renamed ETH_RST
- U1 pad 16: unconnected-(U1-GPIO16-Pad16) -> ETH_QSPI_CS
- U1 pad 17: unconnected-(U1-GPIO17-Pad17) -> ETH_QSPI_CK
- U1 pad 18: unconnected-(U1-GPIO18-Pad18) -> ETH_QSPI_Q0
- U1 pad 19: unconnected-(U1-GPIO19-Pad19) -> ETH_QSPI_Q1
- U1 pad 20: unconnected-(U1-GPIO20-Pad20) -> ETH_QSPI_Q2
- U1 pad 21: unconnected-(U1-GPIO21-Pad21) -> ETH_QSPI_Q3
- U1 pad 33: Net-(J10-SWCLK/TCK) -> Net-(U1-SWCLK)
- U1 pad 34: Net-(J10-SWDIO/TMS) -> Net-(U1-SWDIO)
- U1 pad 35: unconnected-(U1-RUN-Pad35) -> Net-(U1-RUN)
- U1 pad 66: unconnected-(U1-USB_DM-Pad66) -> Net-(U1-USB_DM)
- U1 pad 67: unconnected-(U1-USB_DP-Pad67) -> Net-(U1-USB_DP)
- U1 pad 70: Net-(U1-QSPI_SD3) -> unconnected-(U1-QSPI_SD3-Pad70)
- U1 pad 71: Net-(U1-QSPI_SCLK) -> unconnected-(U1-QSPI_SCLK-Pad71)
- U1 pad 72: Net-(U1-QSPI_SD0) -> unconnected-(U1-QSPI_SD0-Pad72)
- U1 pad 73: Net-(U1-QSPI_SD2) -> unconnected-(U1-QSPI_SD2-Pad73)
- U1 pad 74: Net-(U1-QSPI_SD1) -> unconnected-(U1-QSPI_SD1-Pad74)
- U2 pad 29: Net-(U1-~{QSPI_SS}) -> ETH_QSPI_CS
- U2 pad 30: Net-(U1-QSPI_SCLK) -> ETH_QSPI_CK
- U2 pad 32: Net-(U1-QSPI_SD0) -> ETH_QSPI_Q0
- U2 pad 33: Net-(U1-QSPI_SD1) -> ETH_QSPI_Q1
- U2 pad 34: Net-(U1-QSPI_SD2) -> ETH_QSPI_Q2
- U2 pad 35: Net-(U1-QSPI_SD3) -> ETH_QSPI_Q3

Commit message: Adding power and stuff.
Parts:
- added C27: 100n, Capacitor_SMD:C_0603_1608Metric, F.Cu at (139.2, 107.9)
- added C28: 100n, Capacitor_SMD:C_0603_1608Metric, F.Cu at (139.2, 110.4)
- added C29: 100n, Capacitor_SMD:C_0603_1608Metric, F.Cu at (139.2, 112.9)
- added C30: 100n, Capacitor_SMD:C_0603_1608Metric, F.Cu at (139.2, 115.4)
- added C31: 100n, Capacitor_SMD:C_0603_1608Metric, F.Cu at (139.2, 117.9)
- added C32: 100n, Capacitor_SMD:C_0603_1608Metric, F.Cu at (139.2, 120.4)
- added C33: 100n, Capacitor_SMD:C_0603_1608Metric, F.Cu at (143.2, 107.9)
- added C34: 100n, Capacitor_SMD:C_0603_1608Metric, F.Cu at (143.2, 110.4)
- added C35: 100n, Capacitor_SMD:C_0603_1608Metric, F.Cu at (143.2, 112.9)
- added C36: 100n, Capacitor_SMD:C_0603_1608Metric, F.Cu at (143.2, 115.4)
- added R1: 33, Resistor_SMD:R_0603_1608Metric, F.Cu at (143.2, 117.9)
- added U3: RT6150AGQW, Richtek_RT6150:WDFN-10-1EP_3x3mm_P0.5mm_EP1.8x2.5mm, F.Cu at (214.6, 74.7)
- moved U2 55.1 mm to (204.9, 97.0)
- moved J9 51.8 mm to (186.6, 78.0)
- moved R4 44.8 mm to (193.9, 108.7)
- moved R3 44.8 mm to (193.9, 106.2)
- moved R5 44.8 mm to (193.9, 111.2)
- moved R6 44.8 mm to (193.9, 113.7)
- moved R7 38.4 mm to (197.9, 93.7)
- moved R8 38.4 mm to (197.9, 96.2)
- moved C7 35.4 mm to (185.9, 96.2)
- moved C6 35.4 mm to (185.9, 93.7)
- moved C8 35.4 mm to (185.9, 98.7)
- moved C9 33.6 mm to (185.9, 101.2)
- moved C10 33.6 mm to (185.9, 103.7)
- moved R10 32.0 mm to (197.9, 101.2)
- moved R12 32.0 mm to (197.9, 106.2)
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Connections:
- R18 pad 1: Net-(U1-SWCLK) -> Net-(J10-SWCLK/TCK)
- R18 pad 2: Net-(J10-SWCLK/TCK) -> Net-(U1-SWCLK)
- R19 pad 1: Net-(J10-SWDIO/TMS) -> Net-(U1-SWDIO)
- R19 pad 2: Net-(U1-SWDIO) -> Net-(J10-SWDIO/TMS)

Commit message: WIP.
Parts:
- removed the C26 at (153.4, 101.4)
- removed the J1 at (126.1, 65.5)
- removed the J2 at (126.1, 73.2)
- removed J3: Conn_01x07, Connector_JST:JST_GH_BM07B-GHS-TBT_1x07-1MP_P1.25mm_Vertical
- removed the R13 at (153.4, 103.9)
- removed the R14 at (153.4, 106.4)
- removed the R15 at (153.4, 108.9)
- added C36: 100n, Capacitor_SMD:C_0603_1608Metric, F.Cu at (93.1, 101.5)
- added C37: 47μ/6.3V, Capacitor_SMD:C_0603_1608Metric, F.Cu at (93.1, 104.0)
- added C38: 100n, Capacitor_SMD:C_0603_1608Metric, F.Cu at (143.0, 98.8)
- added C39: 100n, Capacitor_SMD:C_0603_1608Metric, F.Cu at (143.0, 103.3)
- added C40: 100n, Capacitor_SMD:C_0603_1608Metric, F.Cu at (182.3, 80.0)
- added C41: 100n, Capacitor_SMD:C_0603_1608Metric, F.Cu at (182.3, 63.3)
- added C42: 100n, Capacitor_SMD:C_0603_1608Metric, F.Cu at (128.3, 62.5)
- added C43: 100n, Capacitor_SMD:C_0603_1608Metric, F.Cu at (128.3, 45.8)
- added CP1: C_Array_4x0612, AVX_Capacitor_Array:C_Array_4x0612, F.Cu at (128.7, 103.0)
- added CP2: C_Array_4x0612, AVX_Capacitor_Array:C_Array_4x0612, F.Cu at (113.7, 104.5)
- added CP3: C_Array_4x0612, AVX_Capacitor_Array:C_Array_4x0612, F.Cu at (181.1, 88.8)
- added CP4: C_Array_4x0612, AVX_Capacitor_Array:C_Array_4x0612, F.Cu at (181.1, 72.0)
- added CP5: C_Array_4x0612, AVX_Capacitor_Array:C_Array_4x0612, F.Cu at (127.1, 71.3)
- added CP6: C_Array_4x0612, AVX_Capacitor_Array:C_Array_4x0612, F.Cu at (127.1, 54.5)
- added H1: MountingHole, MountingHole:MountingHole_3.2mm_M3_NoCopper, F.Cu at (90.0, 65.0)
- added H2: MountingHole, MountingHole:MountingHole_3.2mm_M3_NoCopper, F.Cu at (90.0, 105.0)
- added H3: MountingHole, MountingHole:MountingHole_3.2mm_M3_NoCopper, F.Cu at (160.0, 65.0)
- added H4: MountingHole, MountingHole:MountingHole_3.2mm_M3_NoCopper, F.Cu at (160.0, 105.0)
- added J9: Conn_01x07, Connector_JST:JST_GH_BM07B-GHS-TBT_1x07-1MP_P1.25mm_Vertical, F.Cu at (119.1, 48.3)
- added JP1: SolderJumper_2_Open, Jumper:SolderJumper-2_P1.3mm_Open_RoundedPad1.0x1.5mm, F.Cu at (132.7, 97.3)
- added JP10: SolderJumper_2_Bridged, Jumper:SolderJumper-2_P1.3mm_Bridged_RoundedPad1.0x1.5mm, F.Cu at (118.9, 74.2)
- added JP11: SolderJumper_2_Open, Jumper:SolderJumper-2_P1.3mm_Open_RoundedPad1.0x1.5mm, F.Cu at (118.9, 53.9)
- added JP12: SolderJumper_2_Bridged, Jumper:SolderJumper-2_P1.3mm_Bridged_RoundedPad1.0x1.5mm, F.Cu at (118.9, 57.5)
- added JP2: SolderJumper_2_Bridged, Jumper:SolderJumper-2_P1.3mm_Bridged_RoundedPad1.0x1.5mm, F.Cu at (132.7, 93.8)
- added JP3: SolderJumper_2_Open, Jumper:SolderJumper-2_P1.3mm_Open_RoundedPad1.0x1.5mm, F.Cu at (132.7, 106.4)
- added JP4: SolderJumper_2_Bridged, Jumper:SolderJumper-2_P1.3mm_Bridged_RoundedPad1.0x1.5mm, F.Cu at (132.7, 102.9)
- added JP5: SolderJumper_2_Open, Jumper:SolderJumper-2_P1.3mm_Open_RoundedPad1.0x1.5mm, F.Cu at (172.9, 88.2)
- added JP6: SolderJumper_2_Bridged, Jumper:SolderJumper-2_P1.3mm_Bridged_RoundedPad1.0x1.5mm, F.Cu at (172.9, 91.7)
- added JP7: SolderJumper_2_Open, Jumper:SolderJumper-2_P1.3mm_Open_RoundedPad1.0x1.5mm, F.Cu at (172.9, 71.4)
- added JP8: SolderJumper_2_Bridged, Jumper:SolderJumper-2_P1.3mm_Bridged_RoundedPad1.0x1.5mm, F.Cu at (172.9, 75.0)
- added JP9: SolderJumper_2_Open, Jumper:SolderJumper-2_P1.3mm_Open_RoundedPad1.0x1.5mm, F.Cu at (118.9, 70.7)
- added L5: 2.2μ, Richtek_RT6150:WDFN-10-1EP_3x3mm_P0.5mm_EP1.8x2.5mm, F.Cu at (141.0, 86.5)
- added R20: 5k6, Resistor_SMD:R_0603_1608Metric, F.Cu at (93.1, 106.5)
- added R21: 10k, Resistor_SMD:R_0603_1608Metric, F.Cu at (93.1, 109.0)
- added R22: 100k, Resistor_SMD:R_0603_1608Metric, F.Cu at (93.1, 111.5)
- added R23: 100k, Resistor_SMD:R_0603_1608Metric, F.Cu at (93.1, 119.0)
- added R24: 487k, Resistor_SMD:R_0603_1608Metric, F.Cu at (93.1, 114.0)
- added R25: 86.6k, Resistor_SMD:R_0603_1608Metric, F.Cu at (93.1, 116.5)
- added R26: 100k, Resistor_SMD:R_0603_1608Metric, F.Cu at (120.8, 104.4)
- added R27: 10k, Resistor_SMD:R_0603_1608Metric, F.Cu at (136.9, 93.3)
- added R28: 100k, Resistor_SMD:R_0603_1608Metric, F.Cu at (105.8, 105.9)
- added R29: 10k, Resistor_SMD:R_0603_1608Metric, F.Cu at (136.9, 102.4)
- added R30: 100k, Resistor_SMD:R_0603_1608Metric, F.Cu at (182.3, 82.5)
- added R31: 10k, Resistor_SMD:R_0603_1608Metric, F.Cu at (182.3, 85.0)
- added R32: 100k, Resistor_SMD:R_0603_1608Metric, F.Cu at (182.3, 65.8)
- added R33: 10k, Resistor_SMD:R_0603_1608Metric, F.Cu at (182.3, 68.3)
- added R34: 100k, Resistor_SMD:R_0603_1608Metric, F.Cu at (128.3, 65.0)
- added R35: 10k, Resistor_SMD:R_0603_1608Metric, F.Cu at (128.3, 67.5)
- added R36: 100k, Resistor_SMD:R_0603_1608Metric, F.Cu at (128.3, 48.3)
- added R37: 10k, Resistor_SMD:R_0603_1608Metric, F.Cu at (128.3, 50.8)
- added RN1: R_Pack04, Resistor_SMD:R_Array_Concave_4x0603, F.Cu at (124.8, 103.1)
- added RN2: R_Pack04, Resistor_SMD:R_Array_Concave_4x0603, F.Cu at (109.8, 104.6)
- added RN3: R_Pack04, Resistor_SMD:R_Array_Concave_4x0603, F.Cu at (177.2, 88.8)
- added RN4: R_Pack04, Resistor_SMD:R_Array_Concave_4x0603, F.Cu at (177.2, 72.1)
- added RN5: R_Pack04, Resistor_SMD:R_Array_Concave_4x0603, F.Cu at (123.2, 71.3)
- added RN6: R_Pack04, Resistor_SMD:R_Array_Concave_4x0603, F.Cu at (123.2, 54.6)
- added U4: 74AHC125, Package_DFN_QFN:DHVQFN-14-1EP_2.5x3mm_P0.5mm_EP1x1.5mm, F.Cu at (116.4, 103.7)
- added U5: 74AHC125, Package_DFN_QFN:DHVQFN-14-1EP_2.5x3mm_P0.5mm_EP1x1.5mm, F.Cu at (101.4, 105.2)
- added U6: 74AHC125, Package_DFN_QFN:DHVQFN-14-1EP_2.5x3mm_P0.5mm_EP1x1.5mm, F.Cu at (168.4, 89.4)
- added U7: 74AHC125, Package_DFN_QFN:DHVQFN-14-1EP_2.5x3mm_P0.5mm_EP1x1.5mm, F.Cu at (168.4, 72.7)
- added U8: 74AHC125, Package_DFN_QFN:DHVQFN-14-1EP_2.5x3mm_P0.5mm_EP1x1.5mm, F.Cu at (114.4, 71.9)
- added U9: 74AHC125, Package_DFN_QFN:DHVQFN-14-1EP_2.5x3mm_P0.5mm_EP1x1.5mm, F.Cu at (114.4, 55.2)
- moved U2 89.0 mm to (117.0, 83.8)
- moved J2 80.8 mm to (106.5, 88.9), turned to 180 degrees
- moved U3 73.2 mm to (141.5, 79.5)
- moved J7 65.5 mm to (173.1, 65.8)
- moved J8 54.5 mm to (119.1, 65.1)
- moved J6 51.6 mm to (173.1, 82.6)
- moved J5 20.1 mm to (106.1, 98.3)
- moved U1 11.2 mm to (129.4, 83.5)
- moved J1 9.75 mm to (157.6, 75.0)
- moved J4 9.73 mm to (121.1, 96.8)
- renumbered C36 to C10, C28 to C13, C27 to C14, C29 to C15, C8 to C16, C7 to C17, C6 to C18, C9 to C19, C10 to C20, C17 to C21, C18 to C22, C19 to C23, C12 to C24, C11 to C25, C20 to C26, C21 to C27, C22 to C28, C13 to C29, C23 to C30, C14 to C31, C24 to C32, C15 to C33, C25 to C34, C16 to C35, C35 to C4, C34 to C5, C33 to C6, C32 to C7, C31 to C8, C30 to C9, J10 to J1, J9 to J2, L3 to L2, L2 to L3, R4 to R10, R3 to R11, R5 to R12, R6 to R13, R7 to R14, R8 to R15, R10 to R16, R9 to R17, R11 to R18, R12 to R19, R20 to R3, R16 to R4, R17 to R5, R22 to R6, R21 to R7, R18 to R8, R19 to R9
Connections:
- net +3.3VA renamed 3V3A
- J1 pad 10: unconnected-(J10-~{RESET}-Pad10) -> Net-(J1-~{RESET})
- J1 pad 9: unconnected-(J10-GNDDetect-Pad9) -> GND
- J4 pad 1: unconnected-(J4-Pin_1-Pad1) -> VSYS
- J4 pad 2: unconnected-(J4-Pin_2-Pad2) -> GND
- J4 pad 3: unconnected-(J4-Pin_3-Pad3) -> +3V3
- J4 pad 4: unconnected-(J4-Pin_4-Pad4) -> Net-(J4-Pin_4)
- J4 pad 5: unconnected-(J4-Pin_5-Pad5) -> Net-(J4-Pin_5)
- J4 pad 6: unconnected-(J4-Pin_6-Pad6) -> Net-(J4-Pin_6)
- J4 pad 7: unconnected-(J4-Pin_7-Pad7) -> Net-(J4-Pin_7)
- J5 pad 1: unconnected-(J5-Pin_1-Pad1) -> VSYS
- J5 pad 2: unconnected-(J5-Pin_2-Pad2) -> GND
- J5 pad 3: unconnected-(J5-Pin_3-Pad3) -> +3V3
- J5 pad 4: unconnected-(J5-Pin_4-Pad4) -> Net-(J5-Pin_4)
- J5 pad 5: unconnected-(J5-Pin_5-Pad5) -> Net-(J5-Pin_5)
- J5 pad 6: unconnected-(J5-Pin_6-Pad6) -> Net-(J5-Pin_6)
- J5 pad 7: unconnected-(J5-Pin_7-Pad7) -> Net-(J5-Pin_7)
- J6 pad 1: unconnected-(J6-Pin_1-Pad1) -> VSYS
- J6 pad 2: unconnected-(J6-Pin_2-Pad2) -> GND
- J6 pad 3: unconnected-(J6-Pin_3-Pad3) -> +3V3
- J6 pad 4: unconnected-(J6-Pin_4-Pad4) -> Net-(J6-Pin_4)
- J6 pad 5: unconnected-(J6-Pin_5-Pad5) -> Net-(J6-Pin_5)
- J6 pad 6: unconnected-(J6-Pin_6-Pad6) -> Net-(J6-Pin_6)
- J6 pad 7: unconnected-(J6-Pin_7-Pad7) -> Net-(J6-Pin_7)
- J7 pad 1: unconnected-(J7-Pin_1-Pad1) -> VSYS
- J7 pad 2: unconnected-(J7-Pin_2-Pad2) -> GND
- J7 pad 3: unconnected-(J7-Pin_3-Pad3) -> +3V3
- J7 pad 4: unconnected-(J7-Pin_4-Pad4) -> Net-(J7-Pin_4)
- J7 pad 5: unconnected-(J7-Pin_5-Pad5) -> Net-(J7-Pin_5)
- J7 pad 6: unconnected-(J7-Pin_6-Pad6) -> Net-(J7-Pin_6)
- J7 pad 7: unconnected-(J7-Pin_7-Pad7) -> Net-(J7-Pin_7)
- J8 pad 1: unconnected-(J8-Pin_1-Pad1) -> VSYS
- J8 pad 2: unconnected-(J8-Pin_2-Pad2) -> GND
- J8 pad 3: unconnected-(J8-Pin_3-Pad3) -> +3V3
- J8 pad 4: unconnected-(J8-Pin_4-Pad4) -> Net-(J8-Pin_4)
- J8 pad 5: unconnected-(J8-Pin_5-Pad5) -> Net-(J8-Pin_5)
- J8 pad 6: unconnected-(J8-Pin_6-Pad6) -> Net-(J8-Pin_6)
- J8 pad 7: unconnected-(J8-Pin_7-Pad7) -> Net-(J8-Pin_7)
- R3 pad 1: Net-(R20-Pad1) -> Net-(J1-~{RESET})
- U1 pad 23: unconnected-(U1-GPIO23-Pad23) -> POWER_SAVE
- U1 pad 25: unconnected-(U1-GPIO24-Pad25) -> VBUS_MONITOR
- U1 pad 39: unconnected-(U1-GPIO31-Pad39) -> BRICKLET_CS_F
- U1 pad 40: unconnected-(U1-GPIO32-Pad40) -> BRICKLET_CS_E
- U1 pad 42: unconnected-(U1-GPIO33-Pad42) -> BRICKLET_CS_D
- U1 pad 43: unconnected-(U1-GPIO34-Pad43) -> BRICKLET_CS_C
- U1 pad 44: unconnected-(U1-GPIO35-Pad44) -> BRICKLET_CS_B
- U1 pad 45: unconnected-(U1-GPIO36-Pad45) -> BRICKLET_MISO
- U1 pad 46: unconnected-(U1-GPIO37-Pad46) -> BRICKLET_CS_A
- U1 pad 47: unconnected-(U1-GPIO38-Pad47) -> BRICKLET_CLK
- U1 pad 48: unconnected-(U1-GPIO39-Pad48) -> BRICKLET_MOSI
- U2 pad 10: +3V3 -> 3V3D
- U2 pad 24: +3V3 -> 3V3D
- U2 pad 36: +3V3 -> 3V3D
- U3 pad 1: unconnected-(U3-VOUT-Pad1) -> +3V3
- U3 pad 10: unconnected-(U3-FB-Pad10) -> Net-(U3-FB)
- U3 pad 11: unconnected-(U3-EP-Pad11) -> GND
- U3 pad 2: unconnected-(U3-LX2-Pad2) -> Net-(U3-LX2)
- U3 pad 3: unconnected-(U3-GND-Pad3) -> GND
- U3 pad 4: unconnected-(U3-LX1-Pad4) -> Net-(U3-LX1)
- U3 pad 5: unconnected-(U3-VIN-Pad5) -> VSYS
- U3 pad 6: unconnected-(U3-EN-Pad6) -> Net-(U3-EN)
- U3 pad 7: unconnected-(U3-PS-Pad7) -> POWER_SAVE
- U3 pad 8: unconnected-(U3-VINA-Pad8) -> VSYS
- U3 pad 9: unconnected-(U3-GND-Pad9) -> GND
Other:
- board outline added: 77 x 47 mm

Commit message: WIP.
Parts:
- added C1: 4.7μ/6.3V, Capacitor_SMD:C_0603_1608Metric, F.Cu at (148.0, 83.3)
- added C11: 4.7μ/6.3V, Capacitor_SMD:C_0603_1608Metric, F.Cu at (148.0, 90.8)
- added C12: 4.7μ/6.3V, Capacitor_SMD:C_0603_1608Metric, F.Cu at (148.0, 93.3)
- added C2: 15p, Capacitor_SMD:C_0603_1608Metric, F.Cu at (148.0, 85.8)
- added C3: 15p, Capacitor_SMD:C_0603_1608Metric, F.Cu at (148.0, 88.3)
- added D1: PMEG6010ELRX, Diode_SMD:Nexperia_CFP3_SOD-123W, F.Cu at (161.4, 83.6)
- added L6: AOTA-B201610S3R3-101-T, Abracon_AOTA_B201610S:L_0806_2016Metric, F.Cu at (137.8, 70.6)
- added P1: USB_C_Plug_USB2.0, Connector_USB:USB_C_Receptacle_GCT_USB4085, F.Cu at (167.8, 119.1)
- added R2: 1k, Resistor_SMD:R_0603_1608Metric, F.Cu at (148.0, 95.8)
- added R38: 5.1k, Resistor_SMD:R_0603_1608Metric, F.Cu at (168.2, 115.5)
- added SW1: SW_Push, Littelfuse_CK_PTS815:SW_SPST_CK_PTS815_Sx250SMTR_LFS, F.Cu at (153.3, 84.4)
- added SW2: SW_Push, Littelfuse_CK_PTS815:SW_SPST_CK_PTS815_Sx250SMTR_LFS, F.Cu at (153.3, 89.1)
- added Y1: ABM8-272-T3, Crystal:Crystal_SMD_Abracon_ABM8G-4Pin_3.2x2.5mm, F.Cu at (152.6, 93.8)
- added Y2: 25MHz, Crystal:Crystal_SMD_Abracon_ABM8G-4Pin_3.2x2.5mm, F.Cu at (161.2, 89.5)
Connections:
- net ETH_INT renamed /WizNet/INT
- net ETH_QSPI_CK renamed /WizNet/QSPI_CLK
- net ETH_QSPI_CS renamed /WizNet/QSPI_CS
- net ETH_QSPI_Q0 renamed /WizNet/QSPI_Q0
- net ETH_QSPI_Q1 renamed /WizNet/QSPI_Q1
- net ETH_QSPI_Q2 renamed /WizNet/QSPI_Q2
- net ETH_QSPI_Q3 renamed /WizNet/QSPI_Q3
- net ETH_RST renamed /WizNet/RST
- R20 pad 1: VBUS -> /Power/V_USB
- R4 pad 1: USB_DN -> Net-(P1-D-)
- R5 pad 1: USB_DP -> Net-(P1-D+)
- U2 pad 10: 3V3D -> +3V3
- U2 pad 24: 3V3D -> +3V3
- U2 pad 36: 3V3D -> +3V3

Commit message: Working on bricklet bus. Kinda like it.
Parts:
- removed C38, C39, C40, C41: 100n, Capacitor_SMD:C_0603_1608Metric
- removed CP1, CP2, CP3, CP4: C_Array_4x0612, AVX_Capacitor_Array:C_Array_4x0612
- removed J4, J5, J6, J7: Conn_01x07, Connector_JST:JST_GH_BM07B-GHS-TBT_1x07-1MP_P1.25mm_Vertical
- removed JP1, JP3, JP5, JP7: SolderJumper_2_Open, Jumper:SolderJumper-2_P1.3mm_Open_RoundedPad1.0x1.5mm
- removed JP2, JP4, JP6, JP8: SolderJumper_2_Bridged, Jumper:SolderJumper-2_P1.3mm_Bridged_RoundedPad1.0x1.5mm
- removed R26, R28, R30, R32: 100k, Resistor_SMD:R_0603_1608Metric
- removed R27, R29, R31, R33: 10k, Resistor_SMD:R_0603_1608Metric
- removed RN1, RN2, RN3, RN4: R_Pack04, Resistor_SMD:R_Array_Concave_4x0603
- removed U4, U5, U6, U7: 74AHC125, Package_DFN_QFN:DHVQFN-14-1EP_2.5x3mm_P0.5mm_EP1x1.5mm
- added C44: 100n, Capacitor_SMD:C_0603_1608Metric, F.Cu at (127.3, 94.3)
- added CP7: C_Array_4x0612, AVX_Capacitor_Array:C_Array_4x0612, F.Cu at (126.1, 103.0)
- added D2: PMEG6010ELRX, Diode_SMD:Nexperia_CFP3_SOD-123W, F.Cu at (113.8, 111.4)
- added J10: Conn_01x07, Connector_JST:JST_GH_BM07B-GHS-TBT_1x07-1MP_P1.25mm_Vertical, F.Cu at (118.1, 96.8)
- added JP13: SolderJumper_2_Open, Jumper:SolderJumper-2_P1.3mm_Open_RoundedPad1.0x1.5mm, F.Cu at (117.9, 102.4)
- added JP14: SolderJumper_2_Bridged, Jumper:SolderJumper-2_P1.3mm_Bridged_RoundedPad1.0x1.5mm, F.Cu at (117.9, 106.0)
- added R39: 100k, Resistor_SMD:R_0603_1608Metric, F.Cu at (127.3, 96.8)
- added R40: 10k, Resistor_SMD:R_0603_1608Metric, F.Cu at (127.3, 99.3)
- added RN7: R_Pack04, Resistor_SMD:R_Array_Concave_4x0603, F.Cu at (122.2, 103.1)
- added U10: 74AHC125, Package_DFN_QFN:DHVQFN-14-1EP_2.5x3mm_P0.5mm_EP1x1.5mm, F.Cu at (113.4, 103.7)
Connections:
- net BRICKLET_CLK renamed /CLK
- JP11 pad 1: BRICKLET_CS_F -> /CS_1
- JP9 pad 1: BRICKLET_CS_E -> /CS_2
- R35 pad 1: BRICKLET_CS_E -> /CS_2
- R37 pad 1: BRICKLET_CS_F -> /CS_1
- U1 pad 39: BRICKLET_CS_F -> unconnected-(U1-GPIO31-Pad39)
- U1 pad 40: BRICKLET_CS_E -> unconnected-(U1-GPIO32-Pad40)
- U1 pad 42: BRICKLET_CS_D -> /CS_3
- U1 pad 43: BRICKLET_CS_C -> /CS_2
- U1 pad 44: BRICKLET_CS_B -> /CS_1
- U1 pad 45: BRICKLET_MISO -> /MOSI
- U1 pad 46: BRICKLET_CS_A -> unconnected-(U1-GPIO37-Pad46)
- U1 pad 48: BRICKLET_MOSI -> /MISO
- U8 pad 1: BRICKLET_CS_E -> /CS_2
- U8 pad 10: BRICKLET_CS_E -> /CS_2
- U8 pad 11: BRICKLET_MISO -> /MISO
- U8 pad 13: BRICKLET_CS_E -> /CS_2
- U8 pad 2: BRICKLET_CS_E -> /CS_2
- U8 pad 4: BRICKLET_CS_E -> /CS_2
- U8 pad 5: BRICKLET_MOSI -> /MOSI
- U9 pad 1: BRICKLET_CS_F -> /CS_1
- U9 pad 10: BRICKLET_CS_F -> /CS_1
- U9 pad 11: BRICKLET_MISO -> /MISO
- U9 pad 13: BRICKLET_CS_F -> /CS_1
- U9 pad 2: BRICKLET_CS_F -> /CS_1
- U9 pad 4: BRICKLET_CS_F -> /CS_1
- U9 pad 5: BRICKLET_MOSI -> /MOSI

Commit message: Starting to look at routing.
Parts:
- removed C16: 100n, Capacitor_SMD:C_0603_1608Metric
- removed R12, R13: 330, Resistor_SMD:R_0603_1608Metric
- added C38: 1n/2kV, Capacitor_SMD:C_0603_1608Metric, F.Cu at (183.0, 86.8)
- added C39: 100n, Capacitor_SMD:C_0603_1608Metric, F.Cu at (183.0, 89.3)
- added D3: RUNNING, Diode_SMD:D_0603_1608Metric, F.Cu at (177.9, 42.5)
- added D4: SERVER GOOD, Diode_SMD:D_0603_1608Metric, F.Cu at (177.9, 45.1)
- added D5: IP GOOD, Diode_SMD:D_0603_1608Metric, F.Cu at (177.9, 47.7)
- added R26: 2.2k, Resistor_SMD:R_0603_1608Metric, F.Cu at (181.9, 42.5)
- added R27: 2.2k, Resistor_SMD:R_0603_1608Metric, F.Cu at (181.9, 45.0)
- added R28: 2.2k, Resistor_SMD:R_0603_1608Metric, F.Cu at (181.9, 47.5)
- added R29: 49.9, Resistor_SMD:R_0603_1608Metric, F.Cu at (115.3, 76.8)
- added R30: 49.9, Resistor_SMD:R_0603_1608Metric, F.Cu at (115.1, 80.5)
- C19: value 19p -> 18p
- C24: value 100n -> 1µ
- L2, L3, L4: value L -> 120Ω
- R14, R15: value 330 -> 49.9
- R4: value 27 -> 27?
- R5: value R -> 85?
- SW1: value SW_Push -> RST
- SW2: value SW_Push -> BOOT
- moved R15 85.6 mm to (115.1, 74.5)
- moved R14 83.9 mm to (115.4, 78.8)
- moved R17 81.0 mm to (117.8, 86.9), turned to -90 degrees
- moved R16 80.2 mm to (119.3, 85.4), turned to -90 degrees
- moved C34 77.7 mm to (118.3, 78.0)
- moved C32 76.9 mm to (118.3, 79.5)
- moved C31 73.2 mm to (119.9, 82.2)
- moved C20 71.6 mm to (116.3, 86.9), turned to -90 degrees
- moved C27 71.4 mm to (121.6, 88.1), turned to 90 degrees
- moved C19 70.8 mm to (117.1, 84.7)
- moved C28 70.7 mm to (123.1, 88.1), turned to 90 degrees
- moved C33 69.1 mm to (123.3, 75.0), turned to -90 degrees
- moved C18 68.7 mm to (118.3, 81.0)
- moved C26 67.8 mm to (124.6, 88.1), turned to 90 degrees
- moved C29 63.9 mm to (126.1, 88.8), turned to 90 degrees
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Connections:
- net VSYS renamed +5V
- C1 pad 1: Net-(U1-VREG_AVDD) -> GND
- C1 pad 2: GND -> Net-(U1-VREG_AVDD)
- C26 pad 1: GND -> GNDA
- C27 pad 1: GND -> GNDA
- C28 pad 1: GND -> GNDA
- C30 pad 1: GND -> GNDA
- C32 pad 1: GND -> GNDA
- C34 pad 1: GND -> GNDA
- J2 pad SH: unconnected-(J2-SHIELD-PadSH)_1 -> Net-(J2-SHIELD)
- R1 pad 1: +3V3 -> Net-(U1-VREG_AVDD)
- R1 pad 2: Net-(U1-VREG_AVDD) -> +3V3
- R10 pad 1: +3V3 -> Net-(J2-LEDY_A)
- R10 pad 2: Net-(J2-LEDY_A) -> +3V3
- R11 pad 1: +3V3 -> Net-(J2-LEDG_A)
- R11 pad 2: Net-(J2-LEDG_A) -> +3V3
- R14 pad 1: Net-(J2-TD-) -> Net-(J2-RD+)
- R15 pad 1: Net-(J2-TD+) -> Net-(J2-RD-)
- U1 pad 77: unconnected-(U1-GPIO0-Pad77) -> Net-(U1-GPIO0)
- U1 pad 78: unconnected-(U1-GPIO1-Pad78) -> Net-(U1-GPIO1)
- U1 pad 79: unconnected-(U1-GPIO2-Pad79) -> Net-(U1-GPIO2)
Routing:
- net Net-(U2-1V2O): vias 0 -> 2
- added copper zone on In2.Cu, net +3V3
- added copper zone on F.Cu, net GND
- added copper zone on In1.Cu, net GND
Other:
- copper layers 2 -> 4

Commit message: Doing some routing.
Parts:
- added R41: 5.1k, Resistor_SMD:R_0603_1608Metric, F.Cu at (166.1, 73.7)
- JP10, JP9, R35: moved to B.Cu
- L5: footprint Richtek_RT6150:WDFN-10-1EP_3x3mm_P0.5mm_EP1.8x2.5mm -> Abracon_AOTA_B201610S:L_0806_2016Metric
- moved C8 56.9 mm to (138.0, 72.3), turned to -90 degrees
- moved R5 56.7 mm to (141.1, 70.7), turned to -90 degrees
- moved R4 53.8 mm to (142.7, 70.7), turned to -90 degrees
- moved Y1 52.5 mm to (142.6, 94.8)
- moved C2 51.7 mm to (140.8, 91.5)
- moved C42 51.2 mm to (115.9, 66.9), turned to -90 degrees
- moved C9 50.3 mm to (149.9, 76.6), turned to 180 degrees
- moved C21 49.3 mm to (152.4, 107.0), turned to 90 degrees
- moved R35 48.4 mm to (115.0, 63.7), turned to 180 degrees
- moved C3 47.4 mm to (144.4, 91.5), turned to 180 degrees
- moved C10 45.3 mm to (150.0, 81.2), turned to 180 degrees
- moved R2 44.7 mm to (143.6, 88.5), turned to 90 degrees
- moved C15 44.5 mm to (134.8, 80.2)
- moved C7 43.0 mm to (141.6, 88.5), turned to 90 degrees
- moved C13 42.4 mm to (150.0, 79.6), turned to 180 degrees
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Connections:
- C38 pad 2: Net-(J2-SHIELD) -> GNDPWR
- CP5 pad 1: Net-(J8-Pin_4) -> Net-(J8-Pin_6)
- CP5 pad 3: Net-(J8-Pin_6) -> Net-(J8-Pin_4)
- CP6 pad 1: Net-(J9-Pin_4) -> Net-(J9-Pin_6)
- CP6 pad 3: Net-(J9-Pin_6) -> Net-(J9-Pin_4)
- CP7 pad 1: Net-(J10-Pin_4) -> Net-(J10-Pin_6)
- CP7 pad 3: Net-(J10-Pin_6) -> Net-(J10-Pin_4)
- J10 pad MP: (no net) -> GND
- J2 pad SH: Net-(J2-SHIELD) -> GNDPWR
- J8 pad MP: (no net) -> GND
- J9 pad MP: (no net) -> GND
- P1 pad A6: Net-(P1-D+) -> Net-(P1-D+-PadA6)
- P1 pad A7: Net-(P1-D-) -> Net-(P1-D--PadA7)
- P1 pad A8: (no net) -> unconnected-(P1-SBU1-PadA8)
- P1 pad B5: unconnected-(P1-VCONN-PadB5) -> Net-(P1-CC2)
- P1 pad B6: (no net) -> Net-(P1-D+-PadA6)
- P1 pad B7: (no net) -> Net-(P1-D--PadA7)
- P1 pad B8: (no net) -> unconnected-(P1-SBU2-PadB8)
- P1 pad SH: unconnected-(P1-SHIELD-PadSH)_2 -> GNDPWR
- R4 pad 1: Net-(P1-D-) -> Net-(P1-D--PadA7)
- R5 pad 1: Net-(P1-D+) -> Net-(P1-D+-PadA6)
- RN5 pad 1: Net-(RN5-R1.1) -> Net-(J8-Pin_7)
- RN5 pad 2: Net-(RN5-R2.1) -> Net-(J8-Pin_6)
- RN5 pad 3: Net-(RN5-R3.1) -> Net-(J8-Pin_5)
- RN5 pad 4: Net-(JP10-A) -> Net-(J8-Pin_4)
- RN5 pad 5: Net-(J8-Pin_4) -> Net-(JP10-A)
- RN5 pad 6: Net-(J8-Pin_5) -> Net-(RN5-R3.2)
- RN5 pad 7: Net-(J8-Pin_6) -> Net-(RN5-R2.2)
- RN5 pad 8: Net-(J8-Pin_7) -> Net-(RN5-R1.2)
- RN6 pad 1: Net-(RN6-R1.1) -> Net-(J9-Pin_7)
- RN6 pad 2: Net-(RN6-R2.1) -> Net-(J9-Pin_6)
- RN6 pad 3: Net-(RN6-R3.1) -> Net-(J9-Pin_5)
- RN6 pad 4: Net-(JP11-B) -> Net-(J9-Pin_4)
- RN6 pad 5: Net-(J9-Pin_4) -> Net-(JP11-B)
- RN6 pad 6: Net-(J9-Pin_5) -> Net-(RN6-R3.2)
- RN6 pad 7: Net-(J9-Pin_6) -> Net-(RN6-R2.2)
- RN6 pad 8: Net-(J9-Pin_7) -> Net-(RN6-R1.2)
- RN7 pad 1: Net-(RN7-R1.1) -> Net-(J10-Pin_7)
- RN7 pad 2: Net-(RN7-R2.1) -> Net-(J10-Pin_6)
- RN7 pad 3: Net-(RN7-R3.1) -> Net-(J10-Pin_5)
- RN7 pad 4: Net-(JP13-B) -> Net-(J10-Pin_4)
- RN7 pad 5: Net-(J10-Pin_4) -> Net-(JP13-B)
- RN7 pad 6: Net-(J10-Pin_5) -> Net-(RN7-R3.2)
- RN7 pad 7: Net-(J10-Pin_6) -> Net-(RN7-R2.2)
- RN7 pad 8: Net-(J10-Pin_7) -> Net-(RN7-R1.2)
- U10 pad 12: Net-(RN7-R1.1) -> Net-(RN7-R1.2)
- U10 pad 6: Net-(RN7-R3.1) -> Net-(RN7-R3.2)
- U10 pad 8: Net-(RN7-R2.1) -> Net-(RN7-R2.2)
- U8 pad 12: Net-(RN5-R1.1) -> Net-(RN5-R1.2)
- U8 pad 6: Net-(RN5-R3.1) -> Net-(RN5-R3.2)
- U8 pad 8: Net-(RN5-R2.1) -> Net-(RN5-R2.2)
- U9 pad 12: Net-(RN6-R1.1) -> Net-(RN6-R1.2)
- U9 pad 6: Net-(RN6-R3.1) -> Net-(RN6-R3.2)
- U9 pad 8: Net-(RN6-R2.1) -> Net-(RN6-R2.2)
- Y2 pad 2: Net-(C20-Pad2) -> GND
- Y2 pad 3: (no net) -> Net-(C20-Pad2)
- Y2 pad 4: (no net) -> GND
Routing:
- net Net-(U1-XIN): track 0.00 -> 11.4 mm
- net +3V3: track 0.00 -> 10.9 mm, vias 0 -> 1
- net +1V1: track 0.00 -> 9.84 mm
- net Net-(J8-Pin_4): track 0.00 -> 7.88 mm, vias 0 -> 2
- net GND: track 0.00 -> 7.80 mm, vias 0 -> 11
- net Net-(J8-Pin_5): track 0.00 -> 6.39 mm, vias 0 -> 2
- net Net-(C3-Pad2): track 0.00 -> 5.68 mm
- net Net-(U1-USB_DP): track 0.00 -> 5.02 mm
- net Net-(J8-Pin_6): track 0.00 -> 4.78 mm, vias 0 -> 2
- net Net-(U1-USB_DM): track 0.00 -> 4.50 mm
- net Net-(RN5-R3.2): track 0.00 -> 3.96 mm
- net Net-(U1-XOUT): track 0.00 -> 2.76 mm
- net Net-(RN5-R2.2): track 0.00 -> 0.80 mm, vias 0 -> 1
Other:
- board text added: "More decoupling caps on RP?"

Commit message: Routing.
Parts:
- moved JP10 23.3 mm to (112.5, 68.2)
- moved JP9 21.5 mm to (115.8, 68.2)
- moved CP5 9.67 mm to (119.2, 64.8)
- moved J8 9.67 mm to (112.8, 60.0)
- moved R34 9.67 mm to (119.2, 67.7)
- moved U8 9.67 mm to (110.0, 65.6)
- moved RN5 9.67 mm to (114.2, 65.8)
- moved C42 7.23 mm to (108.8, 68.5), turned to 0 degrees
- moved R35 5.28 mm to (110.2, 66.0)
- moved C13 0.75 mm to (150.8, 79.6)
Routing:
- net /CS_2: track 0.00 -> 19.6 mm, vias 0 -> 3
- net Net-(RN5-R1.2): track 0.00 -> 12.1 mm, vias 0 -> 2
- net Net-(RN5-R2.2): track 0.80 -> 8.38 mm, vias 1 -> 2
- net GND: track 7.80 -> 15.1 mm, vias 11 -> 25
- net +3V3: track 10.9 -> 17.4 mm, vias 1 -> 3
- net Net-(J8-Pin_5): track 6.39 -> 11.9 mm
- net +1V1: track 9.84 -> 15.0 mm, vias 0 -> 3
- net Net-(JP10-A): track 0.00 -> 3.61 mm, vias 0 -> 1
- net Net-(J8-Pin_7): track 0.00 -> 3.52 mm
- net Net-(JP10-B): track 0.00 -> 2.57 mm, vias 0 -> 1
- net Net-(J8-Pin_6): track 4.78 -> 6.46 mm
- net Net-(J8-Pin_4): track 7.88 -> 9.27 mm
- net /CLK: track 0.00 -> 1.18 mm, vias 0 -> 1
- net /MISO: track 0.00 -> 1.14 mm, vias 0 -> 1
- net /MOSI: track 0.00 -> 0.82 mm, vias 0 -> 1
- added copper zone on F.Cu, net +1V1
- added copper zone on F.Cu, net +3V3
