File: pcb/gateway/gateway2/gateway2.kicad_pcb (KiCad board)
At the start: 4 copper layers, 77 x 47 mm, 104 parts, among them J1 Conn_ARM_JTAG_SWD_10, J2 RJ45_Kycon_G7LX-A88S7-BP-GY, J8 Conn_01x07, P1 USB_C_Plug_USB2.0, SW1 RST, SW2 BOOT, U1 RP2354B, U2 W6300-Q, U3 RT6150AGQW, U8 74AHC125, Y1 ABM8-272-T3, Y2 25MHz

Commit message: Routing on.
Parts:
- U2: footprint Package_QFP:LQFP-48-1EP_7x7mm_P0.5mm_EP3.6x3.6mm_ThermalVias -> Package_QFP:LQFP-48-1EP_7x7mm_P0.5mm_EP3.6x3.6mm
- moved C39 24.4 mm to (114.4, 72.7), turned to -90 degrees
- moved R19 22.9 mm to (119.8, 76.0), turned to -90 degrees
- moved R18 21.2 mm to (118.2, 76.0), turned to 90 degrees
- moved R16 10.2 mm to (120.0, 86.3)
- moved C32 7.51 mm to (117.2, 84.0)
- moved C17 7.26 mm to (114.4, 91.9), turned to 90 degrees
- moved L3 7.01 mm to (123.8, 88.5)
- moved C34 6.07 mm to (117.2, 82.5)
- moved C20 5.70 mm to (118.2, 92.3), turned to 90 degrees
- moved C18 5.41 mm to (116.0, 76.5), turned to -90 degrees
- moved R17 3.75 mm to (121.5, 86.3)
- moved L4 3.07 mm to (119.9, 90.8), turned to 90 degrees
- moved C19 3.07 mm to (116.2, 92.3), turned to 90 degrees
- moved C26 1.99 mm to (124.7, 90.8)
- moved C27 1.99 mm to (123.0, 90.8)
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Connections:
- C17 pad 1: GNDA -> GND
- C18 pad 1: GNDA -> GND
- C26 pad 1: GNDA -> GND
- C27 pad 1: GNDA -> GND
- C28 pad 1: GNDA -> GND
- C30 pad 1: GNDA -> GND
- C32 pad 1: GNDA -> GND
- C34 pad 1: GNDA -> GND
- C39 pad 1: GNDA -> GND
- U2 pad 15: GNDA -> GND
- U2 pad 17: GNDA -> GND
- U2 pad 48: GNDA -> GND
- U2 pad 6: GNDA -> GND
Routing:
- net GND: track 29.8 -> 67.6 mm, vias 45 -> 61
- net Net-(J2-LEDY_K): track 0.00 -> 35.4 mm, vias 0 -> 1
- net 3V3A: track 10.6 -> 41.3 mm, vias 1 -> 8
- net Net-(U2-XSCI): track 0.00 -> 12.5 mm
- net Net-(C17-Pad2): track 0.00 -> 10.7 mm, vias 0 -> 2
- net Net-(C39-Pad2): track 0.00 -> 10.7 mm, vias 0 -> 2
- net Net-(U2-RSET_BG): track 0.00 -> 8.95 mm, vias 0 -> 2
- net Net-(C20-Pad2): track 0.00 -> 6.48 mm
- net 1V2A: track 0.00 -> 6.27 mm
- net Net-(U2-XSCO): track 0.00 -> 4.16 mm
- net Net-(J2-LEDY_A): track 0.00 -> 3.69 mm
- net Net-(U2-1V2O): track 0.00 -> 3.42 mm, vias 2 -> 0
- net +3V3: track 29.4 -> 32.3 mm, vias 11 -> 16
- net Net-(R18-Pad2): track 0.00 -> 1.55 mm
- net 1V2D: track 14.4 -> 15.6 mm
