File: pcb/gateway/gateway2/gateway2.kicad_sch (KiCad schematic)
At the start: 55 parts, among them J1 Conn_01x07, J10 Conn_ARM_JTAG_SWD_10, J2 Conn_01x07, J3 Conn_01x07, J4 Conn_01x07, J5 Conn_01x07, J6 Conn_01x07, J7 Conn_01x07, J8 Conn_01x07, J9 RJ45_Kycon_G7LX-A88S7-BP-GY, U1 RP2354B, U2 W6300-Q, Y1 RP-01G8X7-GS352B, Y2 Crystal

Commit message: Continuing draft. Adding sample projects, datasheets.
Parts:
- added C26: 100n, Capacitor_SMD:C_0603_1608Metric, symbol Device:C
- added D1: D_Schottky, symbol Device:D_Schottky
- added J11: Conn_01x05, symbol Connector_Generic:Conn_01x05
- added R13: 5k6, Resistor_SMD:R_0603_1608Metric, symbol Device:R
- added R14, R22: 10k, Resistor_SMD:R_0603_1608Metric, symbol Device:R
- added R15: 100k, Resistor_SMD:R_0603_1608Metric, symbol Device:R
- added R16: 27, Resistor_SMD:R_0603_1608Metric, symbol Device:R
- added R17: R, Resistor_SMD:R_0603_1608Metric, symbol Device:R
- added R18, R19: 100, Resistor_SMD:R_0603_1608Metric, symbol Device:R
- added R20, R21: 1k, Resistor_SMD:R_0603_1608Metric, symbol Device:R
- added SW1, SW2: SW_Push, symbol Switch:SW_Push
Connections:
- net +3V3: now also R22.1
- net GND: now also C26.1, J11.5 (Pin_5), R14.2, SW1.1, SW2.1
- net at J10.2 (SWDIO/TMS): now also R19.2; no longer U1.34 (SWDIO)
- net at J10.4 (SWCLK/TCK): now also R18.1; no longer U1.33 (SWCLK)
- net ETH_INT: now reaches U1.14 (GPIO15), U2.45 (~{INT})
- net ETH_QSPI_CS: now reaches U1.16 (GPIO16)
- net ETH_QSPI_CS: now also U2.29 (~{CS})
- net ETH_QSPI_CK: now reaches U1.17 (GPIO17)
- net ETH_QSPI_CK: now also U2.30 (SCLK)
- net ETH_QSPI_Q0: now reaches U1.18 (GPIO18)
- net ETH_QSPI_Q0: now also U2.32 (QD0/ADDR0)
- net ETH_QSPI_Q1: now reaches U1.19 (GPIO19)
- net ETH_QSPI_Q1: now also U2.33 (QD1/ADDR1)
- net ETH_QSPI_Q2: now reaches U1.20 (GPIO20)
- net ETH_QSPI_Q2: now also U2.34 (QD2/~{RD})
- net ETH_QSPI_Q3: now reaches U1.21 (GPIO21)
- net ETH_QSPI_Q3: now also U2.35 (QD3/~{WR})
- net ETH_RST: now reaches U1.22 (GPIO22), U2.46 (~{RST})
- net at U1.35 (RUN): now also R20.2
- net at U1.66 (USB_DM): now also R16.2
- net at U1.67 (USB_DP): now also R17.2
- net at U1.70 (QSPI_SD3): no longer U2.35 (QD3/~{WR})
- net at U1.71 (QSPI_SCLK): no longer U2.30 (SCLK)
- net at U1.72 (QSPI_SD0): no longer U2.32 (QD0/ADDR0)
- net at U1.73 (QSPI_SD2): no longer U2.34 (QD2/~{RD})
- net at U1.74 (QSPI_SD1): no longer U2.33 (QD1/ADDR1)
- net at U1.75 (~{QSPI_SS}): now also R21.2, R22.2; no longer U2.29 (~{CS})
- new net: R13.2, R14.1
- new net: R19.1, U1.34 (SWDIO)
- new net: R21.1, SW2.2
- new net: R20.1, SW1.2
- new net: R18.2, U1.33 (SWCLK)
- new net USB_DN: J11.2 (Pin_2), R16.1
- new net USB_DP: J11.3 (Pin_3), R17.1
- new net VBUS: D1.2 (A), J11.1 (Pin_1), R13.1
- new net VSYS: C26.2, D1.1 (K), R15.1
Other:
- note added: "3V3 coverter here"
- note added: "Do I do POE?"
- note added: "GND detect?"
- note added: "POE which lines?"
- moved on the sheet: C1, C2, C3, C4, C5, J10, L1, R1, R2, U1, Y1

Commit message: Adding power and stuff.
Parts:
- removed C10: 18p, Capacitor_SMD:C_0603_1608Metric, symbol Device:C
- removed C11, C12, C13, C14, C15, C16, C17, C18, C19, C20, C21, C22, C23, C24, C25, C26, C6, C7, C8: 100n, Capacitor_SMD:C_0603_1608Metric, symbol Device:C
- removed C9: 19p, Capacitor_SMD:C_0603_1608Metric, symbol Device:C
- removed D1: D_Schottky, symbol Device:D_Schottky
- removed J11: Conn_01x05, symbol Connector_Generic:Conn_01x05
- removed J9: RJ45_Kycon_G7LX-A88S7-BP-GY, Connector_RJ:RJ45_Kycon_G7LX-A88S7-BP-xx_Horizontal, symbol Connector:RJ45_Kycon_G7LX-A88S7-BP-GY
- removed L2, L3, L4: L, Inductor_SMD:L_0603_1608Metric, symbol Device:L
- removed R10: 1M, Resistor_SMD:R_0603_1608Metric, symbol Device:R
- removed R11: 12k, Resistor_SMD:R_0603_1608Metric, symbol Device:R
- removed R12: 300, Resistor_SMD:R_0603_1608Metric, symbol Device:R
- removed R13: 5k6, Resistor_SMD:R_0603_1608Metric, symbol Device:R
- removed R14: 10k, Resistor_SMD:R_0603_1608Metric, symbol Device:R
- removed R15: 100k, Resistor_SMD:R_0603_1608Metric, symbol Device:R
- removed R3, R4, R5, R6, R7, R8: 330, Resistor_SMD:R_0603_1608Metric, symbol Device:R
- removed R9: 0, Resistor_SMD:R_0603_1608Metric, symbol Device:R
- removed U2: W6300-Q, WIZnet_W6300:W6300-Q, symbol WIZnet_W6300:W6300-Q
- removed Y2: Crystal, symbol Device:Crystal
- added C27, C28, C29, C30, C31, C32, C33, C34, C35, C36: 100n, Capacitor_SMD:C_0603_1608Metric, symbol Device:C
- C3: value C -> 4.7μ/6.3V
- R1: value R -> 33; footprint (none) -> Resistor_SMD:R_0603_1608Metric
Connections:
- net +1V1: now also C27.2, C28.2, C29.2
- net +3V3: now also C30.2, C31.2, C32.2, C33.2, C34.2, C35.2, C36.2
- net GND: now also C27.1, C28.1, C29.1, C30.1, C31.1, C32.1, C33.1, C34.1, C35.1, C36.1
- net POWER_SAVE: now reaches U1.23 (GPIO23)
- net VBUS_MONITOR: now reaches U1.25 (GPIO24)
- no-connect marks 8 -> 0
Other:
- added sheet Power (Power.kicad_sch)
- added sheet WizNet (WizNet.kicad_sch)
- note added: ""We found that as the VREG_AVDD only draws around 200 μA, an RC filter of 33 Ω and 4.7 μF is adequate.""
- note added: "Routing this is absolutely crucial!"
- note added: "WizNet pins"
- note removed: "3V3 coverter here"
- note removed: "Do I do POE?"
- note removed: "POE which lines?"
- note removed: "Why this in series?"
- moved on the sheet: C1, C2, C3, C4, C5, J1, J10, L1, R1, R16, R17, R18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

Commit message: WIP.
Parts:
- removed J1, J2, J3, J4, J5, J6, J7, J8: Conn_01x07, Connector_JST:JST_GH_BM07B-GHS-TBT_1x07-1MP_P1.25mm_Vertical, symbol Connector_Generic:Conn_01x07
- added H1, H2, H3, H4: MountingHole, MountingHole:MountingHole_3.2mm_M3_NoCopper, symbol Mechanical:MountingHole
- C1: renamed from C3; footprint (none) -> Capacitor_SMD:C_0603_1608Metric
- C11: renamed from C2; value C -> 4.7μ/6.3V; footprint (none) -> Capacitor_SMD:C_0603_1608Metric
- C12: renamed from C1; value C -> 4.7μ/6.3V; footprint (none) -> Capacitor_SMD:C_0603_1608Metric
- C2: renamed from C4; value C -> 15p; footprint (none) -> Capacitor_SMD:C_0603_1608Metric
- C3: renamed from C5; value C -> 15p; footprint (none) -> Capacitor_SMD:C_0603_1608Metric
- R2: value R -> 1k; footprint (none) -> Resistor_SMD:R_0603_1608Metric
- Y1: value RP-01G8X7-GS352B -> ABM8-272-T3; footprint (none) -> Crystal:Crystal_SMD_Abracon_ABM8G-4Pin_3.2x2.5mm
- renumbered C36 to C10, C28 to C13, C27 to C14, C29 to C15, C35 to C4, C34 to C5, C33 to C6, C32 to C7, C31 to C8, C30 to C9, J10 to J1, R20 to R3, R16 to R4, R17 to R5, R22 to R6, R21 to R7, R18 to R8, R19 to R9
Connections:
- net GND: now also J1.9 (GNDDetect), Y1.2 (G), Y1.4 (G)
- net at J1.10 (~{RESET}): now also R3.1, SW1.2
- net BRICKLET_CS_F: now reaches U1.39 (GPIO31)
- net BRICKLET_CS_E: now reaches U1.40 (GPIO32)
- net BRICKLET_CS_D: now reaches U1.42 (GPIO33)
- net BRICKLET_CS_C: now reaches U1.43 (GPIO34)
- net BRICKLET_CS_B: now reaches U1.44 (GPIO35)
- net BRICKLET_MISO: now reaches U1.45 (GPIO36)
- net BRICKLET_CS_A: now reaches U1.46 (GPIO37)
- net BRICKLET_CLK: now reaches U1.47 (GPIO38)
- net BRICKLET_MOSI: now reaches U1.48 (GPIO39)
- no-connect marks 0 -> 36
Other:
- added sheet BrickletPort1 (Bricklet.kicad_sch)
- added sheet BrickletPort2 (Bricklet.kicad_sch)
- added sheet BrickletPort3 (Bricklet.kicad_sch)
- added sheet BrickletPort4 (Bricklet.kicad_sch)
- added sheet BrickletPort5 (Bricklet.kicad_sch)
- added sheet BrickletPort6 (Bricklet.kicad_sch)
- sheet WizNet ports: added +3V3; removed none
- note added: "External flash for data?"
- moved on the sheet: C1, C10, C11, C12, C13, C14, C15, C2, C3, C4, C5, C6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

Commit message: WIP.
Parts:
- removed L1: L, symbol Device:L
- added L6: AOTA-B201610S3R3-101-T, Abracon_AOTA_B201610S:L_0806_2016Metric, symbol Custom_Passives:L_Polarised
- added P1: USB_C_Plug_USB2.0, Connector_USB:USB_C_Receptacle_GCT_USB4085, symbol Connector:USB_C_Plug_USB2.0
- added R38: 5.1k, Resistor_SMD:R_0603_1608Metric, symbol Device:R
- SW1, SW2: footprint (none) -> Littelfuse_CK_PTS815:SW_SPST_CK_PTS815_Sx250SMTR_LFS
Connections:
- net +1V1: now also L6.1
- net GND: now also P1.A1 (GND), P1.A12 (GND), P1.B1 (GND), P1.B12 (GND), R38.1
- net at U1.63 (VREG_LX): now also L6.2
- net ETH_INT renamed WizNet/INT
- net ETH_QSPI_CK renamed WizNet/QSPI_CLK
- net ETH_QSPI_CS renamed WizNet/QSPI_CS
- net ETH_QSPI_Q0 renamed WizNet/QSPI_Q0
- net ETH_QSPI_Q1 renamed WizNet/QSPI_Q1
- net ETH_QSPI_Q2 renamed WizNet/QSPI_Q2
- net ETH_QSPI_Q3 renamed WizNet/QSPI_Q3
- net ETH_RST renamed WizNet/RST
- net USB_DN: no longer names the net of R4.1
- net USB_DN: now also P1.A7 (D-)
- net USB_DP: no longer names the net of R5.1
- net USB_DP: now also P1.A6 (D+)
- new net: P1.A5 (CC), R38.2
- new net Power/V_USB: P1.A4 (VBUS), P1.A9 (VBUS), P1.B4 (VBUS), P1.B9 (VBUS)
- no-connect marks 36 -> 39
Other:
- sheet Power ports: added +3V3, POWER_SAVE, VBUS_MONITOR, V_AUX, V_USB; removed none
- sheet WizNet ports: added INT, QSPI_CLK, QSPI_CS, QSPI_Q0, QSPI_Q1, QSPI_Q2, QSPI_Q3, RST; removed none
- note added: "Fix those pins"
- note removed: "WizNet pins"
- moved on the sheet: C11, C12

Commit message: Working on bricklet bus. Kinda like it.
Connections:
- net BRICKLET_CLK renamed CLK
- net BRICKLET_CS_A: no longer names the net of U1.46 (GPIO37)
- net BRICKLET_CS_B renamed CS_1
- net BRICKLET_CS_C renamed CS_2
- net BRICKLET_CS_D renamed CS_3
- net BRICKLET_CS_E: no longer names the net of U1.40 (GPIO32)
- net BRICKLET_CS_F: no longer names the net of U1.39 (GPIO31)
- net BRICKLET_MISO renamed MOSI
- net BRICKLET_MOSI renamed MISO
- no-connect marks 39 -> 42
Other:
- removed sheet BrickletPort4
- removed sheet BrickletPort5
- removed sheet BrickletPort6
- sheet BrickletPort1 ports: added none; removed GND
- sheet BrickletPort2 ports: added none; removed GND
- sheet BrickletPort3 ports: added none; removed GND

Commit message: Starting to look at routing.
Parts:
- added D3: RUNNING, Diode_SMD:D_0603_1608Metric, symbol Device:LED
- added D4: SERVER GOOD, Diode_SMD:D_0603_1608Metric, symbol Device:LED
- added D5: IP GOOD, Diode_SMD:D_0603_1608Metric, symbol Device:LED
- added R26, R27, R28: 2.2k, Resistor_SMD:R_0603_1608Metric, symbol Device:R
- R4: value 27 -> 27?
- R5: value R -> 85?
- SW1: value SW_Push -> RST
- SW2: value SW_Push -> BOOT
Connections:
- net +3V3: now also R1.2; no longer R1.1
- net GND: now also C1.1, D3.1 (K), D4.1 (K), D5.1 (K); no longer C1.2
- net at U1.77 (GPIO0): now also R26.1
- net at U1.78 (GPIO1): now also R28.1
- net at U1.79 (GPIO2): now also R27.1
- new net: C1.2, R1.1, U1.61 (VREG_AVDD)
- new net: D5.2 (A), R28.2
- new net: D3.2 (A), R26.2
- new net: D4.2 (A), R27.2
- no-connect marks 42 -> 39
Other:
- sheet Power ports: added +5V; removed none
- note added: "Decoupling caps"
- note added: "Do I do POE?"
- note removed: "GND detect?"
- moved on the sheet: C1, C10, C11, C12, C13, C14, C15, C2, C3, C4, C5, C6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

Commit message: Doing some routing.
Parts:
- added C38: 1n/2kV, Capacitor_SMD:C_0603_1608Metric, symbol Device:C
- added R41: 5.1k, Resistor_SMD:R_0603_1608Metric, symbol Device:R
- P1: symbol Connector:USB_C_Plug_USB2.0 -> Connector:USB_C_Receptacle_USB2.0_16P
Connections:
- net GND: now also C38.1, R41.1
- net at P1.A7 (D-), R4.1: now also P1.B7 (D-)
- net at P1.A6 (D+), R5.1: now also P1.B6 (D+)
- net at P1.B5 (CC2): now also R41.2
- net GNDPWR: now reaches P1.SH (SHIELD)
- net GNDPWR: now also C38.2
Other:
- sheet WizNet ports: added GND_SHIELD; removed none
- note added: "It is unclear how WizNet connects shield GNDs RJ45<->USB"
- note added: "Need to understand this grounding"
- note removed: "Fix those pins"
- moved on the sheet: R38

Commit message: WIP.
Parts:
- removed L6: AOTA-B201610S3R3-101-T, Abracon_AOTA_B201610S:L_0806_2016Metric, symbol Custom_Passives:L_Polarised
- added L1: L, Inductor_SMD:L_Abracon_AOTA-B201610S, symbol Device:L_Polarised
Connections:
- net +1V1: now also L1.1
- net at U1.63 (VREG_LX): now also L1.2
- net USB_D-: now reaches P1.A7 (D-), P1.B7 (D-), R4.1
- net USB_D+: now reaches P1.A6 (D+), P1.B6 (D+), R5.1
Other:
- removed sheet BrickletPort1
- removed sheet BrickletPort3
