File: pcb/gateway/gateway2/gateway2.kicad_sch (KiCad schematic)
At the start: 44 parts, among them J1 Conn_ARM_JTAG_SWD_10, P1 USB_C_Plug_USB2.0, SW1 RST, SW2 BOOT, U1 RP2354B, Y1 ABM8-272-T3

Commit message: Moving stuff to proper library.
Parts:
- L1: value L -> 3.3µ
- SW1, SW2: footprint Littelfuse_CK_PTS815:SW_SPST_CK_PTS815_Sx250SMTR_LFS -> Button_Switch_SMD:SW_SPST_CK_PTS815_Sx250SMTR_LFS
Changed lines of the file:
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@@
 			)
 		)
-		(property "Footprint" "Littelfuse_CK_PTS815:SW_SPST_CK_PTS815_Sx250SMTR_LFS"
+		(property "Footprint" "Button_Switch_SMD:SW_SPST_CK_PTS815_Sx250SMTR_LFS"
 			(at 154.94 120.65 0)
 			(hide yes)
@@
 			)
 		)
-		(property "Footprint" "Littelfuse_CK_PTS815:SW_SPST_CK_PTS815_Sx250SMTR_LFS"
+		(property "Footprint" "Button_Switch_SMD:SW_SPST_CK_PTS815_Sx250SMTR_LFS"
 			(at 154.94 102.87 0)
 			(hide yes)
@@
 			)
 		)
-		(property "Value" "L"
-			(at 219.71 78.3231 0)
-			(show_name no)
-			(do_not_autoplace no)
+		(property "Value" "3.3µ"
+			(at 216.154 81.788 90)
+			(show_name no)
+			(do_not_autoplace no)

Commit message: Cross-routing Wiznet SPI.
Parts:
- added C16: 100n, Capacitor_SMD:C_0603_1608Metric, symbol Device:C
Connections:
- net +3V3: now also C16.2
- net GND: now also C16.1
Changed lines of the file:
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@@
 	)
 	(junction
+		(at 387.35 92.71)
+		(diameter 0)
+		(color 0 0 0 0)
+	)
+	(junction
 		(at 381 92.71)
 		(diameter 0)
@@
 	)
 	(junction
+		(at 387.35 102.87)
+		(diameter 0)
+		(color 0 0 0 0)
+	)
+	(junction
 		(at 219.71 71.12)
 		(diameter 0)
@@
 	(wire
 		(pts
+			(xy 387.35 102.87) (xy 393.7 102.87)
+		)
+		(stroke
+			(width 0)
+			(type default)
+		)
+	)
+	(wire
+		(pts
 			(xy 368.3 101.6) (xy 368.3 102.87)
 		)
@@
 	(wire
 		(pts
+			(xy 393.7 93.98) (xy 393.7 92.71)
+		)
+		(stroke
+			(width 0)
+			(type default)
+		)
+	)
+	(wire
+		(pts
 			(xy 55.88 120.65) (xy 58.42 120.65)
 		)
@@
 		)
 	)
+	(wire
+		(pts
+			(xy 393.7 92.71) (xy 387.35 92.71)
+		)
+		(stroke
+			(width 0)
+			(type default)
+		)
+	)
 	(bus
 		(pts
@@
 	(wire
 		(pts
+			(xy 393.7 101.6) (xy 393.7 102.87)
+		)
+		(stroke
+			(width 0)
+			(type default)
+		)
+	)
+	(wire
+		(pts
 			(xy 134.62 158.75) (xy 138.43 158.75)
 		)
@@
 					(unit 1)
 				)
+			)
+		)
+	)
+	(symbol
+		(lib_id "Device:C")
+		(at 393.7 97.79 180)
+		(unit 1)
+		(body_style 1)
+		(exclude_from_sim no)
+		(in_bom yes)
+		(on_board yes)
+		(in_pos_files yes)
+		(dnp no)
+		(property "Reference" "C16"
+			(at 389.636 95.758 0)
+			(show_name no)
+			(do_not_autoplace no)
+			(effects
+				(font
+					(size 1.27 1.27)
+				)
+				(justify right)
+			)
+		)
+		(property "Value" "100n"
+			(at 388.62 100.076 0)
+			(show_name no)
+			(do_not_autoplace no)
+			(effects
+				(font
+					(size 1.27 1.27)
+				)
+				(justify right)
+			)
+		)
+		(property "Footprint" "Capacitor_SMD:C_0603_1608Metric"
+			(at 392.7348 93.98 0)
+			(hide yes)
+			(show_name no)
+			(do_not_autoplace no)
+			(effects
+				(font
+					(size 1.27 1.27)
+				)
+			)
+		)
+		(property "Datasheet" ""
+			(at 393.7 97.79 0)
+			(hide yes)
+			(show_name no)
+			(do_not_autoplace no)
+			(effects
+				(font
+					(size 1.27 1.27)
+				)
+			)
+		)
+		(property "Description" "Unpolarized capacitor"
+			(at 393.7 97.79 0)
+			(hide yes)
+			(show_name no)
+			(do_not_autoplace no)
+			(effects
+				(font
+					(size 1.27 1.27)
+				)
+			)
+		)
+		(pin "2"
+		)
+		(pin "1"
+		)
+		(instances
+			(project "gateway2"
+				(path "/1800ee7d-fb6b-47f6-b72a-2ea19411a9d6"
+					(reference "C16")
+					(unit 1)
+				)

Commit message: Routing some more.
Parts:
- R4: value 27? -> 27
- R5: value 85? -> 27
Changed lines of the file:
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@@
 			)
 		)
-		(property "Value" "27?"
+		(property "Value" "27"
 			(at 181.61 115.57 90)
 			(show_name no)
@@
 			)
 		)
-		(property "Value" "85?"
+		(property "Value" "27"
 			(at 181.61 118.11 90)
 			(show_name no)

Commit message: Trying to fit 6 bricklet connectors.
Other:
- added sheet BrickletPort1 (Bricklet.kicad_sch)
- added sheet BrickletPort3 (Bricklet.kicad_sch)
- added sheet BrickletPort4 (Bricklet.kicad_sch)
- added sheet BrickletPort5 (Bricklet.kicad_sch)
- added sheet BrickletPort6 (Bricklet.kicad_sch)

Commit message: Still routing.
Connections:
- net CS_1: now also U1.43 (GPIO34); no longer U1.44 (GPIO35)
- net CS_2: now also U1.42 (GPIO33); no longer U1.43 (GPIO34)
- net CS_3: now also U1.44 (GPIO35); no longer U1.42 (GPIO33)
- net CS_4: now also U1.38 (GPIO30)
- net CS_5: now also U1.39 (GPIO31)
- net CS_6: now also U1.40 (GPIO32)
- no-connect marks 39 -> 35
Other:
- sheet Power ports: added none; removed V_AUX
Changed lines of the file:
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@@
 	)
 	(junction
-		(at 299.72 170.18)
+		(at 299.72 165.1)
 		(diameter 0)
 		(color 0 0 0 0)
@@
 	)
 	(no_connect
-		(at 237.49 168.91)
-	)
-	(no_connect
 		(at 237.49 110.49)
 	)
@@
 	)
 	(no_connect
-		(at 237.49 173.99)
-	)
-	(no_connect
 		(at 55.88 128.27)
 	)
@@
 	)
 	(no_connect
-		(at 237.49 171.45)
-	)
-	(no_connect
 		(at 186.69 135.89)
 	)
@@
 	)
 	(no_connect
-		(at 93.98 88.9)
-	)
-	(no_connect
 		(at 237.49 100.33)
 	)
@@
 	)
 	(bus_entry
+		(at 255.27 166.37)
+		(size -2.54 2.54)
+		(stroke
+			(width 0)
+			(type default)
+		)
+	)
+	(bus_entry
 		(at 350.52 204.47)
 		(size 2.54 2.54)
@@
 	)
 	(bus_entry
+		(at 255.27 168.91)
+		(size -2.54 2.54)
+		(stroke
+			(width 0)
+			(type default)
+		)
+	)
+	(bus_entry
 		(at 299.72 228.6)
 		(size 2.54 2.54)
@@
 	)
 	(bus_entry
+		(at 255.27 171.45)
+		(size -2.54 2.54)
+		(stroke
+			(width 0)
+			(type default)
+		)
+	)
+	(bus_entry
 		(at 299.72 223.52)
 		(size 2.54 2.54)
@@
 	(wire
 		(pts
+			(xy 237.49 173.99) (xy 252.73 173.99)
+		)
+		(stroke
+			(width 0)
+			(type default)
+		)
+	)
+	(wire
+		(pts
 			(xy 120.65 87.63) (xy 114.3 87.63)
 		)
@@
 	(bus
 		(pts
-			(xy 255.27 170.18) (xy 255.27 196.85)
+			(xy 255.27 165.1) (xy 255.27 196.85)
 		)
 		(stroke
@@
 	(wire
 		(pts
+			(xy 237.49 168.91) (xy 252.73 168.91)
+		)
+		(stroke
+			(width 0)
+			(type default)
+		)
+	)
+	(wire
+		(pts
 			(xy 368.3 101.6) (xy 368.3 102.87)
 		)
@@
 	(bus
 		(pts
-			(xy 255.27 170.18) (xy 299.72 170.18)
+			(xy 255.27 165.1) (xy 299.72 165.1)
 		)
 		(stroke
@@
 	(bus
 		(pts
-			(xy 350.52 170.18) (xy 350.52 232.41)
+			(xy 350.52 165.1) (xy 350.52 232.41)
 		)
 		(stroke
@@
 	(bus
 		(pts
-			(xy 299.72 170.18) (xy 350.52 170.18)
+			(xy 299.72 165.1) (xy 350.52 165.1)
 		)
 		(stroke
@@
 	(wire
 		(pts
+			(xy 237.49 171.45) (xy 252.73 171.45)
+		)
+		(stroke
+			(width 0)
+			(type default)
+		)
+	)
+	(wire
+		(pts
 			(xy 374.65 64.77) (xy 368.3 64.77)
 		)
@@
 		)
 	)
-	(bus
+	(wire
 		(pts
-			(xy 299.72 170.18) (xy 299.72 232.41)
+			(xy 302.26 209.55) (xy 314.96 209.55)
 		)
 		(stroke
@@
 	(wire
 		(pts
-			(xy 302.26 209.55) (xy 314.96 209.55)
+			(xy 374.65 92.71) (xy 374.65 93.98)
 		)
 		(stroke
@@
 	(wire
 		(pts
-			(xy 374.65 92.71) (xy 374.65 93.98)
+			(xy 158.75 146.05) (xy 157.48 146.05)
 		)
 		(stroke
@@
 		)
 	)
-	(wire
+	(bus
 		(pts
-			(xy 158.75 146.05) (xy 157.48 146.05)
+			(xy 299.72 165.1) (xy 299.72 232.41)
 		)
 		(stroke
@@
 		)
 	)
-	(label "CS_3"
+	(label "CS_2"
 		(at 240.03 176.53 0)
 		(effects
@@
 		)
 	)
-	(label "CS_1"
+	(label "CS_3"
 		(at 240.03 181.61 0)
 		(effects
@@
 		)
 	)
+	(label "CS_4"
+		(at 240.03 168.91 0)
+		(effects
+			(font
+				(size 1.27 1.27)
+			)
+			(justify left bottom)
+		)
+	)
 	(label "CS_3"
 		(at 306.07 226.06 0)
@@
 	)
 	(label "{BrickletBus}"
-		(at 270.51 170.18 0)
+		(at 270.51 165.1 0)
 		(effects
 			(font
@@
 		)
 	)
-	(label "CS_2"
+	(label "CS_1"
 		(at 240.03 179.07 0)
 		(effects
@@
 		)
 	)
+	(label "CS_5"
+		(at 240.03 171.45 0)
+		(effects
+			(font
+				(size 1.27 1.27)
+			)
+			(justify left bottom)
+		)
+	)
+	(label "CS_6"
+		(at 240.03 173.99 0)
+		(effects
+			(font
+				(size 1.27 1.27)
+			)
+			(justify left bottom)
+		)
+	)
 	(label "CS_2"
 		(at 306.07 201.93 0)
@@
 			)
 		)
-		(pin "V_AUX" input
-			(at 93.98 88.9 180)
-			(effects
-				(font
-					(size 1.27 1.27)
-				)
-				(justify left)
-			)
-		)

Commit message: Walking through DRC.
Connections:
- net at U1.77 (GPIO0): now also R28.1; no longer R26.1
- net at U1.78 (GPIO1): now also R27.1; no longer R28.1
- net at U1.79 (GPIO2): now also R26.1; no longer R27.1
Other:
- moved on the sheet: D3, D4, D5, R26, R27, R28

Commit message: Preparing for manufactoring.
Other:
- company: (none) -> ${COMPANY}
- title: (none) -> ${TITLE}
Changed lines of the file:
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@@
 	(generator_version "10.0")
 	(paper "A3")
+	(title_block
+		(title "${TITLE}")
+		(rev "${VERSION}")
+		(company "${COMPANY}")
+	)
 	(text "Decoupling caps"
 		(exclude_from_sim no)

Commit message: Adding some forgotten things: ground hook, power indication LEDs, etc.
Parts:
- added D6: 5V, Diode_SMD:D_0603_1608Metric, symbol Device:LED
- added D7: 3.3V, Diode_SMD:D_0603_1608Metric, symbol Device:LED
- added R31, R32: 2.2k, Resistor_SMD:R_0603_1608Metric, symbol Device:R
- added TP1: TestPoint, TestPoint:TestPoint_Keystone_5019_Miniature, symbol Connector:TestPoint
Connections:
- net +3V3: now also R32.1
- net +5V: now also R31.1
- net GND: now also D6.1 (K), D7.1 (K), TP1.1
- new net: D6.2 (A), R31.2
- new net: D7.2 (A), R32.2
