File: pcb/gateway/gateway2/WizNet.kicad_sch (KiCad schematic)
At the start: 36 parts, among them J9 RJ45_Kycon_G7LX-A88S7-BP-GY, U2 W6300-Q, Y2 Crystal

Commit message: WIP.
Parts:
- Y2: value Crystal -> 25MHz; footprint (none) -> Crystal:Crystal_SMD_Abracon_ABM8G-4Pin_3.2x2.5mm
- renumbered C8 to C16, C7 to C17, C6 to C18, C9 to C19, C10 to C20, C17 to C21, C18 to C22, C19 to C23, C12 to C24, C11 to C25, C20 to C26, C21 to C27, C22 to C28, C13 to C29, C23 to C30, C14 to C31, C24 to C32, C15 to C33, C25 to C34, C16 to C35, J9 to J2, L3 to L2, L2 to L3, R4 to R10, R3 to R11, R5 to R12, R6 to R13, R7 to R14, R8 to R15, R10 to R16, R9 to R17, R11 to R18, R12 to R19
Connections:
- net +3.3VA renamed 3V3A
- net +3V3 renamed 3V3D
- no-connect marks 8 -> 16
Other:
- note added: "Add LEDS"
- note added: "Join GNDs?"

Commit message: WIP.
Connections:
- net ETH_INT renamed INT
- net ETH_QSPI_CK renamed QSPI_CLK
- net ETH_QSPI_CS renamed QSPI_CS
- net ETH_QSPI_Q0 renamed QSPI_Q0
- net ETH_QSPI_Q1 renamed QSPI_Q1
- net ETH_QSPI_Q2 renamed QSPI_Q2
- net ETH_QSPI_Q3 renamed QSPI_Q3
- net ETH_RST renamed RST
Changed lines of the file:
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@@
 	(wire
 		(pts
-			(xy 218.44 91.44) (xy 220.98 91.44)
+			(xy 218.44 91.44) (xy 228.6 91.44)
 		)
 		(stroke
@@
 	(wire
 		(pts
-			(xy 218.44 101.6) (xy 220.98 101.6)
+			(xy 218.44 101.6) (xy 228.6 101.6)
 		)
 		(stroke
@@
 	(wire
 		(pts
-			(xy 218.44 93.98) (xy 220.98 93.98)
+			(xy 218.44 93.98) (xy 228.6 93.98)
 		)
 		(stroke
@@
 	(wire
 		(pts
-			(xy 218.44 114.3) (xy 220.98 114.3)
+			(xy 218.44 114.3) (xy 228.6 114.3)
 		)
 		(stroke
@@
 	(wire
 		(pts
-			(xy 218.44 99.06) (xy 220.98 99.06)
+			(xy 218.44 99.06) (xy 228.6 99.06)
 		)
 		(stroke
@@
 	(wire
 		(pts
-			(xy 218.44 111.76) (xy 220.98 111.76)
+			(xy 218.44 111.76) (xy 228.6 111.76)
 		)
 		(stroke
@@
 	(wire
 		(pts
-			(xy 218.44 109.22) (xy 220.98 109.22)
-		)
-		(stroke
-			(width 0)
-			(type default)
-		)
-	)
-	(wire
-		(pts
-			(xy 218.44 106.68) (xy 220.98 106.68)
-		)
-		(stroke
-			(width 0)
-			(type default)
-		)
-	)
-	(global_label "ETH_QSPI_Q1"
-		(shape input)
-		(at 220.98 109.22 0)
-		(fields_autoplaced yes)
+			(xy 218.44 109.22) (xy 228.6 109.22)
+		)
+		(stroke
+			(width 0)
+			(type default)
+		)
+	)
+	(wire
+		(pts
+			(xy 218.44 106.68) (xy 228.6 106.68)
+		)
+		(stroke
+			(width 0)
+			(type default)
+		)
+	)
+	(hierarchical_label "INT"
+		(shape output)
+		(at 228.6 93.98 0)
 		(effects
 			(font
@@
 			(justify left)
 		)
-		(property "Intersheetrefs" "${INTERSHEET_REFS}"
-			(at 236.3023 109.22 0)
-			(hide yes)
-			(show_name no)
-			(do_not_autoplace no)
-			(effects
-				(font
-					(size 1.27 1.27)
-				)
-				(justify left)
-			)
-		)
-	)
-	(global_label "ETH_RST"
+	)
+	(hierarchical_label "RST"
 		(shape input)
-		(at 220.98 91.44 0)
-		(fields_autoplaced yes)
+		(at 228.6 91.44 0)
 		(effects
 			(font
@@
 			(justify left)
 		)
-		(property "Intersheetrefs" "${INTERSHEET_REFS}"
-			(at 231.827 91.44 0)
-			(hide yes)
-			(show_name no)
-			(do_not_autoplace no)
-			(effects
-				(font
-					(size 1.27 1.27)
-				)
-				(justify left)
-			)
-		)
-	)
-	(global_label "ETH_INT"
-		(shape input)
-		(at 220.98 93.98 0)
-		(fields_autoplaced yes)
+	)
+	(hierarchical_label "QSPI_Q2"
+		(shape bidirectional)
+		(at 228.6 111.76 0)
 		(effects
 			(font
@@
 			(justify left)
 		)
-		(property "Intersheetrefs" "${INTERSHEET_REFS}"
-			(at 231.2828 93.98 0)
-			(hide yes)
-			(show_name no)
-			(do_not_autoplace no)
-			(effects
-				(font
-					(size 1.27 1.27)
-				)
-				(justify left)
-			)
-		)
-	)
-	(global_label "ETH_QSPI_CK"
+	)
+	(hierarchical_label "QSPI_CS"
 		(shape input)
-		(at 220.98 99.06 0)
-		(fields_autoplaced yes)
+		(at 228.6 101.6 0)
 		(effects
 			(font
@@
 			(justify left)
 		)
-		(property "Intersheetrefs" "${INTERSHEET_REFS}"
-			(at 236.3023 99.06 0)
-			(hide yes)
-			(show_name no)
-			(do_not_autoplace no)
-			(effects
-				(font
-					(size 1.27 1.27)
-				)
-				(justify left)
-			)
-		)
-	)
-	(global_label "ETH_QSPI_Q0"
+	)
+	(hierarchical_label "QSPI_CLK"
 		(shape input)
-		(at 220.98 106.68 0)
-		(fields_autoplaced yes)
+		(at 228.6 99.06 0)
 		(effects
 			(font
@@
 			(justify left)
 		)
-		(property "Intersheetrefs" "${INTERSHEET_REFS}"
-			(at 236.3023 106.68 0)
-			(hide yes)
-			(show_name no)
-			(do_not_autoplace no)
-			(effects
-				(font
-					(size 1.27 1.27)
-				)
-				(justify left)
-			)
-		)
-	)
-	(global_label "ETH_QSPI_Q2"
-		(shape input)
-		(at 220.98 111.76 0)
-		(fields_autoplaced yes)
+	)
+	(hierarchical_label "QSPI_Q0"
+		(shape bidirectional)
+		(at 228.6 106.68 0)
 		(effects
 			(font
@@
 			(justify left)
 		)
-		(property "Intersheetrefs" "${INTERSHEET_REFS}"
-			(at 236.3023 111.76 0)
-			(hide yes)
-			(show_name no)
-			(do_not_autoplace no)
-			(effects
-				(font
-					(size 1.27 1.27)
-				)
-				(justify left)
-			)
-		)
-	)
-	(global_label "ETH_QSPI_Q3"
-		(shape input)
-		(at 220.98 114.3 0)
-		(fields_autoplaced yes)
+	)
+	(hierarchical_label "QSPI_Q3"
+		(shape bidirectional)
+		(at 228.6 114.3 0)
 		(effects
 			(font
@@
 			)
 			(justify left)
-		)
-		(property "Intersheetrefs" "${INTERSHEET_REFS}"
-			(at 236.3023 114.3 0)
-			(hide yes)
-			(show_name no)
-			(do_not_autoplace no)
-			(effects
-				(font
-					(size 1.27 1.27)
-				)
-				(justify left)
-			)
-		)
-	)
-	(global_label "ETH_QSPI_CS"
-		(shape input)
-		(at 220.98 101.6 0)
-		(fields_autoplaced yes)
-		(effects
-			(font
-				(size 1.27 1.27)
-			)
-			(justify left)
-		)
-		(property "Intersheetrefs" "${INTERSHEET_REFS}"
-			(at 236.2418 101.6 0)
-			(hide yes)
-			(show_name no)
-			(do_not_autoplace no)
-			(effects
-				(font
-					(size 1.27 1.27)
-				)
-				(justify left)
-			)
 		)
 	)
@@
 		)
 	)
+	(hierarchical_label "QSPI_Q1"
+		(shape bidirectional)
+		(at 228.6 109.22 0)
+		(effects
+			(font
+				(size 1.27 1.27)
+			)
+			(justify left)
+		)
+	)

Commit message: Starting to look at routing.
Parts:
- removed C16: 100n, Capacitor_SMD:C_0603_1608Metric, symbol Device:C
- removed R12, R13: 330, Resistor_SMD:R_0603_1608Metric, symbol Device:R
- added C38: 1n/2kV, Capacitor_SMD:C_0603_1608Metric, symbol Device:C
- added C39: 100n, Capacitor_SMD:C_0603_1608Metric, symbol Device:C
- added JP1: SolderJumper_2_Bridged, symbol Jumper:SolderJumper_2_Bridged
- added R29, R30: 49.9, Resistor_SMD:R_0603_1608Metric, symbol Device:R
- C19: value 19p -> 18p
- C24: value 100n -> 1µ
- L2, L3, L4: value L -> 120Ω; MPN (none) -> MPZ1608S121ATDH5
- R14, R15: value 330 -> 49.9
Connections:
- net 3V3D: now also R10.2, R11.2; no longer R10.1, R11.1
- net GND: now also C38.1, JP1.1 (A); no longer C26.1, C27.1, C28.1, C30.1, C32.1, C34.1
- net GNDA: now also C26.1, C27.1, C28.1, C30.1, C32.1, C34.1, C39.1, JP1.2 (B)
- net at J2.6 (RD-), U2.4 (RXIN): now also R15.1
- net at J2.1 (TD+), U2.2 (TXOP): now also R29.1; no longer R15.1
- net at J2.2 (TD-), U2.1 (TXON): now also R30.1; no longer R14.1
- net at J2.3 (RD+), U2.5 (RXIP): now also R14.1
- net at J2.12 (LEDY_A): now also R10.1; no longer R10.2
- net at J2.14 (LEDG_A): now also R11.1; no longer R11.2
- net at J2.SH (SHIELD): now also C38.2
- new net: C39.2, R29.2, R30.2
- no-connect marks 16 -> 15
Other:
- note added: "Decoupling caps"
- note added: "Need to understand this grounding"
- note removed: "Add LEDS"
- note removed: "Join GNDs?"
- moved on the sheet: C17, C18, C19, C20, C21, C22, C23, C24, C25, C26, C27, C28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

Commit message: Doing some routing.
Parts:
- removed C38: 1n/2kV, Capacitor_SMD:C_0603_1608Metric, symbol Device:C
- Y2: symbol Device:Crystal -> Device:Crystal_GND24
Connections:
- net GND: now also Y2.2 (G), Y2.4 (G)
- net at C20.2, R17.2: now also Y2.3; no longer Y2.2
- net GND_SHIELD: now reaches J2.SH (SHIELD)
Other:
- note removed: "Need to understand this grounding"
Changed lines of the file:
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@@
 		)
 	)
-	(text "Need to understand this grounding"
-		(exclude_from_sim no)
-		(at 46.99 69.596 0)
-		(effects
-			(font
-				(size 1.27 1.27)
-				(color 255 0 0 1)
-			)
-		)
-	)
 	(junction
 		(at 71.12 162.56)
@@
 	(wire
 		(pts
+			(xy 43.18 58.42) (xy 55.88 58.42)
+		)
+		(stroke
+			(width 0)
+			(type default)
+		)
+	)
+	(wire
+		(pts
 			(xy 138.43 101.6) (xy 138.43 102.87)
 		)
@@
 	(wire
 		(pts
-			(xy 44.45 58.42) (xy 55.88 58.42)
-		)
-		(stroke
-			(width 0)
-			(type default)
-		)
-	)
-	(wire
-		(pts
 			(xy 128.27 162.56) (xy 128.27 165.1)
 		)
@@
 	(wire
 		(pts
-			(xy 44.45 60.96) (xy 44.45 58.42)
-		)
-		(stroke
-			(width 0)
-			(type default)
-		)
-	)
-	(wire
-		(pts
 			(xy 204.47 27.94) (xy 198.12 27.94)
 		)
@@
 	(wire
 		(pts
+			(xy 189.23 124.46) (xy 189.23 132.08)
+		)
+		(stroke
+			(width 0)
+			(type default)
+		)
+	)
+	(wire
+		(pts
 			(xy 223.52 123.19) (xy 223.52 125.73)
 		)
@@
 	(wire
 		(pts
-			(xy 44.45 68.58) (xy 44.45 71.12)
-		)
-		(stroke
-			(width 0)
-			(type default)
-		)
-	)
-	(wire
-		(pts
 			(xy 201.93 120.65) (xy 201.93 118.11)
 		)
@@
 		)
 	)
+	(hierarchical_label "GND_SHIELD"
+		(shape input)
+		(at 43.18 58.42 180)
+		(effects
+			(font
+				(size 1.27 1.27)
+			)
+			(justify right)
+		)
+	)
 	(hierarchical_label "INT"
 		(shape output)
@@
 	(symbol
 		(lib_id "power:GND")
-		(at 44.45 71.12 0)
-		(mirror y)
-		(unit 1)
-		(body_style 1)
-		(exclude_from_sim no)
-		(in_bom yes)
-		(on_board yes)
-		(in_pos_files yes)
-		(dnp no)
-		(fields_autoplaced yes)
-		(property "Reference" "#PWR056"
-			(at 44.45 77.47 0)
-			(hide yes)
-			(show_name no)
-			(do_not_autoplace no)
-			(effects
-				(font
-					(size 1.27 1.27)
-				)
-			)
-		)
-		(property "Value" "GND"
-			(at 44.45 76.2 0)
-			(show_name no)
-			(do_not_autoplace no)
-			(effects
-				(font
-					(size 1.27 1.27)
-				)
-			)
-		)
-		(property "Footprint" ""
-			(at 44.45 71.12 0)
-			(hide yes)
-			(show_name no)
-			(do_not_autoplace no)
-			(effects
-				(font
-					(size 1.27 1.27)
-				)
-			)
-		)
-		(property "Datasheet" ""
-			(at 44.45 71.12 0)
-			(hide yes)
-			(show_name no)
-			(do_not_autoplace no)
-			(effects
-				(font
-					(size 1.27 1.27)
-				)
-			)
-		)
-		(property "Description" "Power symbol creates a global label with name \"GND\" , ground"
-			(at 44.45 71.12 0)
-			(hide yes)
-			(show_name no)
-			(do_not_autoplace no)
-			(effects
-				(font
-					(size 1.27 1.27)
-				)
-			)
-		)
-		(pin "1"
-		)
-		(instances
-			(project "gateway2"
-				(path "/1800ee7d-fb6b-47f6-b72a-2ea19411a9d6/a278b076-21e1-4166-b8d0-c689877d5f24"
-					(reference "#PWR056")
-					(unit 1)
-				)
-			)
-		)
-	)
-	(symbol
-		(lib_id "power:GND")
 		(at 44.45 175.26 0)
 		(unit 1)
@@
 		(in_pos_files yes)
 		(dnp no)
-		(fields_autoplaced yes)
 		(property "Reference" "C19"
-			(at 190.5 125.7299 0)
+			(at 194.31 124.968 0)
 			(show_name no)
 			(do_not_autoplace no)
@@
 		)
 		(property "Value" "18p"
-			(at 190.5 128.2699 0)
+			(at 194.056 129.032 0)
 			(show_name no)
 			(do_not_autoplace no)
@@
 	)
 	(symbol
-		(lib_id "Device:Crystal")
+		(lib_id "Device:Crystal_GND24")
 		(at 189.23 119.38 0)
 		(mirror y)
@@
 		(in_pos_files yes)
 		(dnp no)
-		(fields_autoplaced yes)
 		(property "Reference" "Y2"
-			(at 189.23 111.76 0)
+			(at 189.23 119.38 90)
 			(show_name no)
 			(do_not_autoplace no)
@@
 		)
 		(property "Value" "25MHz"
-			(at 189.23 114.3 0)
+			(at 189.23 115.57 0)
 			(show_name no)
 			(do_not_autoplace no)
@@
 			)
 		)
-		(property "Description" "Two pin crystal"
+		(property "Description" "Four pin crystal, GND on pins 2 and 4"
 			(at 189.23 119.38 0)
 			(hide yes)
@@
 		(pin "1"
 		)
+		(pin "4"
+		)
+		(pin "3"
+		)
 		(instances
 			(project "gateway2"
@@
 		(in_pos_files yes)
 		(dnp no)
-		(fields_autoplaced yes)
 		(property "Reference" "R17"
-			(at 181.61 111.7599 0)
+			(at 182.118 115.062 90)
 			(show_name no)
 			(do_not_autoplace no)
@@
 		)
 		(property "Value" "0"
-			(at 181.61 114.2999 0)
+			(at 184.15 113.792 90)
 			(show_name no)
 			(do_not_autoplace no)
@@
 		(in_pos_files yes)
 		(dnp no)
-		(fields_autoplaced yes)
 		(property "Reference" "R16"
-			(at 189.23 101.6 90)
+			(at 189.23 105.918 90)
 			(show_name no)
 			(do_not_autoplace no)
@@
 		)
 		(property "Value" "1M"
-			(at 189.23 104.14 90)
+			(at 189.23 107.95 90)
 			(show_name no)
 			(do_not_autoplace no)
@@
 		(in_pos_files yes)
 		(dnp no)
-		(fields_autoplaced yes)
 		(property "Reference" "C20"
-			(at 180.34 125.7299 0)
+			(at 184.15 124.968 0)
 			(show_name no)
 			(do_not_autoplace no)
@@
 		)
 		(property "Value" "18p"
-			(at 180.34 128.2699 0)
+			(at 183.896 129.032 0)
 			(show_name no)
 			(do_not_autoplace no)
@@
 					(unit 1)
 				)
-			)
-		)
-	)
-	(symbol
-		(lib_id "Device:C")
-		(at 44.45 64.77 180)
-		(unit 1)
-		(body_style 1)
-		(exclude_from_sim no)
-		(in_bom yes)
-		(on_board yes)
-		(in_pos_files yes)
-		(dnp no)
-		(fields_autoplaced yes)
-		(property "Reference" "C38"
-			(at 48.26 63.4999 0)
-			(show_name no)
-			(do_not_autoplace no)
-			(effects
-				(font
-					(size 1.27 1.27)
-				)
-				(justify right)
-			)
-		)
-		(property "Value" "1n/2kV"
-			(at 48.26 66.0399 0)
-			(show_name no)
-			(do_not_autoplace no)
-			(effects
-				(font
-					(size 1.27 1.27)
-				)
-				(justify right)
-			)
-		)
-		(property "Footprint" "Capacitor_SMD:C_0603_1608Metric"
-			(at 43.4848 60.96 0)
-			(hide yes)
-			(show_name no)
-			(do_not_autoplace no)
-			(effects
-				(font
-					(size 1.27 1.27)
-				)
-			)
-		)
-		(property "Datasheet" ""
-			(at 44.45 64.77 0)
-			(hide yes)
-			(show_name no)
-			(do_not_autoplace no)
-			(effects
-				(font
-					(size 1.27 1.27)
-				)
-			)
-		)
-		(property "Description" "Unpolarized capacitor"
-			(at 44.45 64.77 0)
-			(hide yes)
-			(show_name no)
-			(do_not_autoplace no)
-			(effects
-				(font
-					(size 1.27 1.27)
-				)
-			)
-		)
-		(pin "2"
-		)
-		(pin "1"
-		)
-		(instances
-			(project "gateway2"
-				(path "/1800ee7d-fb6b-47f6-b72a-2ea19411a9d6/a278b076-21e1-4166-b8d0-c689877d5f24"
-					(reference "C38")
-					(unit 1)
-				)

Commit message: WIP.
Parts:
- U2: footprint WIZnet_W6300:W6300-Q -> Package_QFP:LQFP-48-1EP_7x7mm_P0.5mm_EP3.6x3.6mm_ThermalVias
Changed lines of the file:
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@@
 			)
 		)
-		(property "Footprint" "WIZnet_W6300:W6300-Q"
+		(property "Footprint" "Package_QFP:LQFP-48-1EP_7x7mm_P0.5mm_EP3.6x3.6mm_ThermalVias"
 			(at 220.98 92.71 0)
 			(hide yes)

Commit message: Fighting ethernet rounting.
Connections:
- net ETH_TD_N: now reaches J2.6 (RD-), R15.1, U2.4 (RXIN)
- net ETH_TD_P: now reaches J2.3 (RD+), R14.1, U2.5 (RXIP)
- net ETH_RD_P: now reaches J2.2 (TD-), R30.1, U2.1 (TXON)
- net ETH_RD_N: now reaches J2.1 (TD+), R29.1, U2.2 (TXOP)
Changed lines of the file:
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@@
+		)
+	)
+	(label "ETH_TD_P"
+		(at 191.77 80.01 0)
+		(effects
+			(font
+				(size 1.27 1.27)
+			)
+			(justify left bottom)
+		)
+	)
+	(label "ETH_TD_N"
+		(at 191.77 82.55 0)
+		(effects
+			(font
+				(size 1.27 1.27)
+			)
+			(justify left bottom)
+		)
+	)
+	(label "ETH_RD_P"
+		(at 191.77 74.93 0)
+		(effects
+			(font
+				(size 1.27 1.27)
+			)
+			(justify left bottom)
+		)
+	)
+	(label "ETH_RD_N"
+		(at 191.77 72.39 0)
+		(effects
+			(font
+				(size 1.27 1.27)
+			)
+			(justify left bottom)
 		)
 	)

Commit message: Routing on.
Parts:
- removed JP1: SolderJumper_2_Bridged, symbol Jumper:SolderJumper_2_Bridged
Connections:
- net GNDA is gone; now on net GND: C17.1, C18.1, C26.1, C27.1, C28.1, C30.1, C32.1, C34.1, C39.1, U2.15 (GNDA), U2.17 (GNDA), U2.48 (GNDA), U2.6 (GNDA)
Changed lines of the file:
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@@
-	(wire
-		(pts
-			(xy 67.31 173.99) (xy 71.12 173.99)
-		)
-		(stroke
-			(width 0)
-			(type default)
-		)
-	)
 	(wire
 		(pts
@@
 	(wire
 		(pts
-			(xy 54.61 173.99) (xy 57.15 173.99)
+			(xy 54.61 173.99) (xy 71.12 173.99)
 		)
 		(stroke
@@
 					(unit 1)
 				)
-			)
-		)
-	)
-	(symbol
-		(lib_id "Jumper:SolderJumper_2_Bridged")
-		(at 62.23 173.99 0)
-		(unit 1)
-		(body_style 1)
-		(exclude_from_sim no)
-		(in_bom no)
-		(on_board yes)
-		(in_pos_files yes)
-		(dnp no)
-		(property "Reference" "JP1"
-			(at 62.23 176.53 0)
-			(show_name no)
-			(do_not_autoplace no)
-			(effects
-				(font
-					(size 1.27 1.27)
-				)
-			)
-		)
-		(property "Value" "SolderJumper_2_Bridged"
-			(at 62.23 170.18 0)
-			(hide yes)
-			(show_name no)
-			(do_not_autoplace no)
-			(effects
-				(font
-					(size 1.27 1.27)
-				)
-			)
-		)
-		(property "Footprint" ""
-			(at 62.23 173.99 0)
-			(hide yes)
-			(show_name no)
-			(do_not_autoplace no)
-			(effects
-				(font
-					(size 1.27 1.27)
-				)
-			)
-		)
-		(property "Datasheet" ""
-			(at 62.23 180.34 0)
-			(hide yes)
-			(show_name no)
-			(do_not_autoplace no)
-			(effects
-				(font
-					(size 1.27 1.27)
-				)
-			)
-		)
-		(property "Description" "Solder Jumper, 2-pole, closed/bridged"
-			(at 62.23 179.07 0)
-			(hide yes)
-			(show_name no)
-			(do_not_autoplace no)
-			(effects
-				(font
-					(size 1.27 1.27)
-				)
-			)
-		)
-		(pin "2"
-		)
-		(pin "1"
-		)
-		(instances
-			(project "gateway2"
-				(path "/1800ee7d-fb6b-47f6-b72a-2ea19411a9d6/a278b076-21e1-4166-b8d0-c689877d5f24"
-					(reference "JP1")
-					(unit 1)
-				)

Commit message: Wiznet power routing is mostly done.
Parts:
- added C44: 100n, Capacitor_SMD:C_0603_1608Metric, symbol Device:C
Connections:
- net 1V2A: now also C44.2
- net GND: now also C44.1
Changed lines of the file:
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@@
 	)
 	(junction
+		(at 219.71 27.94)
+		(diameter 0)
+		(color 0 0 0 0)
+	)
+	(junction
 		(at 71.12 162.56)
 		(diameter 0)
@@
 	)
 	(junction
+		(at 214.63 36.83)
+		(diameter 0)
+		(color 0 0 0 0)
+	)
+	(junction
 		(at 119.38 81.28)
 		(diameter 0)
@@
 	(wire
 		(pts
+			(xy 219.71 27.94) (xy 214.63 27.94)
+		)
+		(stroke
+			(width 0)
+			(type default)
+		)
+	)
+	(wire
+		(pts
 			(xy 119.38 69.85) (xy 119.38 73.66)
 		)
@@
 	(wire
 		(pts
+			(xy 214.63 36.83) (xy 219.71 36.83)
+		)
+		(stroke
+			(width 0)
+			(type default)
+		)
+	)
+	(wire
+		(pts
 			(xy 96.52 76.2) (xy 133.35 76.2)
 		)
@@
 	(wire
 		(pts
-			(xy 220.98 27.94) (xy 214.63 27.94)
+			(xy 220.98 27.94) (xy 219.71 27.94)
 		)
 		(stroke
@@
 	(wire
 		(pts
+			(xy 219.71 27.94) (xy 219.71 29.21)
+		)
+		(stroke
+			(width 0)
+			(type default)
+		)
+	)
+	(wire
+		(pts
 			(xy 194.31 123.19) (xy 194.31 119.38)
 		)
@@
 					(unit 1)
 				)
+			)
+		)
+	)
+	(symbol
+		(lib_id "Device:C")
+		(at 219.71 33.02 180)
+		(unit 1)
+		(body_style 1)
+		(exclude_from_sim no)
+		(in_bom yes)
+		(on_board yes)
+		(in_pos_files yes)
+		(dnp no)
+		(property "Reference" "C44"
+			(at 215.646 31.242 0)
+			(show_name no)
+			(do_not_autoplace no)
+			(effects
+				(font
+					(size 1.27 1.27)
+				)
+				(justify right)
+			)
+		)
+		(property "Value" "100n"
+			(at 214.63 35.306 0)
+			(show_name no)
+			(do_not_autoplace no)
+			(effects
+				(font
+					(size 1.27 1.27)
+				)
+				(justify right)
+			)
+		)
+		(property "Footprint" "Capacitor_SMD:C_0603_1608Metric"
+			(at 218.7448 29.21 0)
+			(hide yes)
+			(show_name no)
+			(do_not_autoplace no)
+			(effects
+				(font
+					(size 1.27 1.27)
+				)
+			)
+		)
+		(property "Datasheet" ""
+			(at 219.71 33.02 0)
+			(hide yes)
+			(show_name no)
+			(do_not_autoplace no)
+			(effects
+				(font
+					(size 1.27 1.27)
+				)
+			)
+		)
+		(property "Description" "Unpolarized capacitor"
+			(at 219.71 33.02 0)
+			(hide yes)
+			(show_name no)
+			(do_not_autoplace no)
+			(effects
+				(font
+					(size 1.27 1.27)
+				)
+			)
+		)
+		(pin "2"
+		)
+		(pin "1"
+		)
+		(instances
+			(project "gateway2"
+				(path "/1800ee7d-fb6b-47f6-b72a-2ea19411a9d6/a278b076-21e1-4166-b8d0-c689877d5f24"
+					(reference "C44")
+					(unit 1)
+				)
