File: pcb/gateway/gateway2/WizNet.kicad_sch (KiCad schematic)
At the start: 37 parts, among them J2 RJ45_Kycon_G7LX-A88S7-BP-GY, U2 W6300-Q, Y2 25MHz

Commit message: Routing some more.
Parts:
- U2: footprint Package_QFP:LQFP-48-1EP_7x7mm_P0.5mm_EP3.6x3.6mm_ThermalVias -> Package_QFP:LQFP-48-1EP_7x7mm_P0.5mm_EP3.6x3.6mm
Changed lines of the file:
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@@
 			)
 		)
-		(property "Footprint" "Package_QFP:LQFP-48-1EP_7x7mm_P0.5mm_EP3.6x3.6mm_ThermalVias"
+		(property "Footprint" "Package_QFP:LQFP-48-1EP_7x7mm_P0.5mm_EP3.6x3.6mm"
 			(at 220.98 92.71 0)
 			(hide yes)

Commit message: Preparing for manufactoring.
Other:
- company: (none) -> ${COMPANY}
- title: (none) -> ${TITLE}
Changed lines of the file:
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@@
 	(generator_version "10.0")
 	(paper "A4")
+	(title_block
+		(title "${TITLE}")
+		(rev "${VERSION}")
+		(company "${COMPANY}")
+	)
 	(text "Decoupling caps"
 		(exclude_from_sim no)
