File: pcb/gateway/gateway2/Bricklet.kicad_sch (KiCad schematic)
At the start: 9 parts, among them J4 Conn_01x07, U4 74AHC125

Commit message: Working on bricklet bus. Kinda like it.
Parts:
- JP13: renamed from JP1; now not fitted
- renumbered C38 to C44, CP1 to CP7, J4 to J10, JP2 to JP14, R26 to R39, R27 to R40, RN1 to RN7, U4 to U10

Commit message: Starting to look at routing.
Other:
- note added: "Decoupling caps"
Changed lines of the file:
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@@
+		)
+	)
+	(text "Decoupling caps"
+		(exclude_from_sim no)
+		(at 256.794 85.344 0)
+		(effects
+			(font
+				(size 1.27 1.27)
+			)
 		)
 	)

Commit message: Doing some routing.
Parts:
- J10: symbol Connector_Generic:Conn_01x07 -> Connector_Generic_MountingPin:Conn_01x07_MountingPin
Connections:
- net GND: now also J10.MP (MountPin)
- net at CP7.2, J10.5 (Pin_5), R39.1: now also RN7.3 (R3.1); no longer RN7.6 (R3.2)
- net at JP13.2 (B), JP14.1 (A): now also RN7.5 (R4.2); no longer RN7.4 (R4.1)
- net at J10.7 (Pin_7): now also RN7.1 (R1.1); no longer RN7.8 (R1.2)
- net at U10.12 (4A): now also RN7.8 (R1.2); no longer RN7.1 (R1.1)
- net at RN7.2 (R2.1): now also CP7.1, J10.6 (Pin_6); no longer U10.8 (3Y)
- net at U10.6 (2Y): now also RN7.6 (R3.2); no longer RN7.3 (R3.1)
- new net: CP7.3, J10.4 (Pin_4), RN7.4 (R4.1)
- new net: RN7.7 (R2.2), U10.8 (3Y)
Other:
- moved on the sheet: RN7
Changed lines of the file:
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@@
 	)
 	(junction
-		(at 134.62 102.87)
+		(at 134.62 97.79)
 		(diameter 0)
 		(color 0 0 0 0)
@@
 	)
 	(junction
+		(at 139.7 102.87)
+		(diameter 0)
+		(color 0 0 0 0)
+	)
+	(junction
 		(at 156.21 97.79)
 		(diameter 0)
@@
 	)
 	(junction
-		(at 139.7 97.79)
+		(at 137.16 100.33)
 		(diameter 0)
 		(color 0 0 0 0)
@@
 	)
 	(junction
-		(at 137.16 100.33)
-		(diameter 0)
-		(color 0 0 0 0)
-	)
-	(junction
 		(at 193.04 97.79)
 		(diameter 0)
@@
 	(wire
 		(pts
-			(xy 109.22 102.87) (xy 134.62 102.87)
-		)
-		(stroke
-			(width 0)
-			(type default)
-		)
-	)
-	(wire
-		(pts
 			(xy 119.38 88.9) (xy 119.38 86.36)
 		)
@@
 	(wire
 		(pts
-			(xy 134.62 102.87) (xy 134.62 109.22)
-		)
-		(stroke
-			(width 0)
-			(type default)
-		)
-	)
-	(wire
-		(pts
 			(xy 171.45 78.74) (xy 181.61 78.74)
 		)
@@
 	(wire
 		(pts
+			(xy 137.16 100.33) (xy 137.16 109.22)
+		)
+		(stroke
+			(width 0)
+			(type default)
+		)
+	)
+	(wire
+		(pts
 			(xy 181.61 77.47) (xy 181.61 91.44)
 		)
@@
 	(wire
 		(pts
-			(xy 134.62 102.87) (xy 144.78 102.87)
-		)
-		(stroke
-			(width 0)
-			(type default)
-		)
-	)
-	(wire
-		(pts
-			(xy 139.7 97.79) (xy 144.78 97.79)
+			(xy 109.22 102.87) (xy 139.7 102.87)
+		)
+		(stroke
+			(width 0)
+			(type default)
+		)
+	)
+	(wire
+		(pts
+			(xy 109.22 97.79) (xy 134.62 97.79)
 		)
 		(stroke
@@
 	(wire
 		(pts
+			(xy 134.62 97.79) (xy 144.78 97.79)
+		)
+		(stroke
+			(width 0)
+			(type default)
+		)
+	)
+	(wire
+		(pts
 			(xy 179.07 118.11) (xy 181.61 118.11)
 		)
@@
 	(wire
 		(pts
-			(xy 139.7 97.79) (xy 139.7 109.22)
-		)
-		(stroke
-			(width 0)
-			(type default)
-		)
-	)
-	(wire
-		(pts
 			(xy 119.38 100.33) (xy 137.16 100.33)
 		)
@@
 	(wire
 		(pts
+			(xy 134.62 97.79) (xy 134.62 109.22)
+		)
+		(stroke
+			(width 0)
+			(type default)
+		)
+	)
+	(wire
+		(pts
 			(xy 113.03 83.82) (xy 113.03 90.17)
 		)
@@
 	(wire
 		(pts
+			(xy 139.7 102.87) (xy 139.7 109.22)
+		)
+		(stroke
+			(width 0)
+			(type default)
+		)
+	)
+	(wire
+		(pts
 			(xy 165.1 107.95) (xy 171.45 107.95)
 		)
@@
 	(wire
 		(pts
+			(xy 104.14 110.49) (xy 104.14 113.03)
+		)
+		(stroke
+			(width 0)
+			(type default)
+		)
+	)
+	(wire
+		(pts
+			(xy 139.7 102.87) (xy 144.78 102.87)
+		)
+		(stroke
+			(width 0)
+			(type default)
+		)
+	)
+	(wire
+		(pts
 			(xy 256.54 97.79) (xy 256.54 99.06)
 		)
@@
 	(wire
 		(pts
-			(xy 109.22 97.79) (xy 139.7 97.79)
-		)
-		(stroke
-			(width 0)
-			(type default)
-		)
-	)
-	(wire
-		(pts
 			(xy 168.91 97.79) (xy 171.45 97.79)
 		)
@@
 	(wire
 		(pts
+			(xy 137.16 100.33) (xy 144.78 100.33)
+		)
+		(stroke
+			(width 0)
+			(type default)
+		)
+	)
+	(wire
+		(pts
 			(xy 179.07 116.84) (xy 179.07 118.11)
 		)
@@
 		(pts
 			(xy 184.15 116.84) (xy 184.15 118.11)
-		)
-		(stroke
-			(width 0)
-			(type default)
-		)
-	)
-	(wire
-		(pts
-			(xy 137.16 100.33) (xy 144.78 100.33)
-		)
-		(stroke
-			(width 0)
-			(type default)
-		)
-	)
-	(wire
-		(pts
-			(xy 137.16 100.33) (xy 137.16 109.22)
 		)
 		(stroke
@@
 	)
 	(symbol
-		(lib_id "Connector_Generic:Conn_01x07")
+		(lib_id "power:GND")
+		(at 104.14 113.03 0)
+		(unit 1)
+		(body_style 1)
+		(exclude_from_sim no)
+		(in_bom yes)
+		(on_board yes)
+		(in_pos_files yes)
+		(dnp no)
+		(fields_autoplaced yes)
+		(property "Reference" "#PWR078"
+			(at 104.14 119.38 0)
+			(hide yes)
+			(show_name no)
+			(do_not_autoplace no)
+			(effects
+				(font
+					(size 1.27 1.27)
+				)
+			)
+		)
+		(property "Value" "GND"
+			(at 104.14 118.11 0)
+			(show_name no)
+			(do_not_autoplace no)
+			(effects
+				(font
+					(size 1.27 1.27)
+				)
+			)
+		)
+		(property "Footprint" ""
+			(at 104.14 113.03 0)
+			(hide yes)
+			(show_name no)
+			(do_not_autoplace no)
+			(effects
+				(font
+					(size 1.27 1.27)
+				)
+			)
+		)
+		(property "Datasheet" ""
+			(at 104.14 113.03 0)
+			(hide yes)
+			(show_name no)
+			(do_not_autoplace no)
+			(effects
+				(font
+					(size 1.27 1.27)
+				)
+			)
+		)
+		(property "Description" "Power symbol creates a global label with name \"GND\" , ground"
+			(at 104.14 113.03 0)
+			(hide yes)
+			(show_name no)
+			(do_not_autoplace no)
+			(effects
+				(font
+					(size 1.27 1.27)
+				)
+			)
+		)
+		(pin "1"
+		)
+		(instances
+			(project "gateway2"
+				(path "/1800ee7d-fb6b-47f6-b72a-2ea19411a9d6/2270f938-9e88-4822-9195-66f8ec9fd89f"
+					(reference "#PWR078")
+					(unit 1)
+				)
+				(path "/1800ee7d-fb6b-47f6-b72a-2ea19411a9d6/48086788-2dae-4fa8-b688-a98b4725ecdb"
+					(reference "#PWR080")
+					(unit 1)
+				)
+				(path "/1800ee7d-fb6b-47f6-b72a-2ea19411a9d6/fe7ca88c-2b6f-471d-ace9-d3d6a951e95f"
+					(reference "#PWR079")
+					(unit 1)
+				)
+			)
+		)
+	)
+	(symbol
+		(lib_id "Connector_Generic_MountingPin:Conn_01x07_MountingPin")
 		(at 104.14 97.79 0)
 		(mirror y)
@@
 			)
 		)
-		(property "Description" "Generic connector, single row, 01x07, script generated (kicad-library-utils/schlib/autogen/connector/)"
+		(property "Description" "Generic connectable mounting pin connector, single row, 01x07, script generated (kicad-library-utils/schlib/autogen/connector/)"
 			(at 104.14 97.79 0)
 			(hide yes)
@@
 		)
 		(pin "2"
+		)
+		(pin "MP"
 		)
 		(instances
@@
 	(symbol
 		(lib_id "Device:R_Pack04")
-		(at 149.86 100.33 90)
+		(at 149.86 100.33 270)
+		(mirror x)
 		(unit 1)
 		(body_style 1)

Commit message: WIP.
Parts:
- renumbered C44 to C42, CP7 to CP5, J10 to J8, JP14 to JP10, JP13 to JP9, R39 to R34, R40 to R35, RN7 to RN5, U10 to U8
Changed lines of the file:
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@@
 		(dnp no)
 		(fields_autoplaced yes)
-		(property "Reference" "R39"
+		(property "Reference" "R34"
 			(at 121.92 91.4399 0)
 			(show_name no)
@@
 		(instances
 			(project "gateway2"
-				(path "/1800ee7d-fb6b-47f6-b72a-2ea19411a9d6/2270f938-9e88-4822-9195-66f8ec9fd89f"
-					(reference "R39")
-					(unit 1)
-				)
-				(path "/1800ee7d-fb6b-47f6-b72a-2ea19411a9d6/48086788-2dae-4fa8-b688-a98b4725ecdb"
-					(reference "R36")
-					(unit 1)
-				)
 				(path "/1800ee7d-fb6b-47f6-b72a-2ea19411a9d6/fe7ca88c-2b6f-471d-ace9-d3d6a951e95f"
 					(reference "R34")
@@
 		(dnp yes)
 		(fields_autoplaced yes)
-		(property "Reference" "JP13"
+		(property "Reference" "JP9"
 			(at 163.83 83.82 0)
 			(show_name no)
@@
 		(instances
 			(project "gateway2"
-				(path "/1800ee7d-fb6b-47f6-b72a-2ea19411a9d6/2270f938-9e88-4822-9195-66f8ec9fd89f"
-					(reference "JP13")
-					(unit 1)
-				)
-				(path "/1800ee7d-fb6b-47f6-b72a-2ea19411a9d6/48086788-2dae-4fa8-b688-a98b4725ecdb"
-					(reference "JP11")
-					(unit 1)
-				)
 				(path "/1800ee7d-fb6b-47f6-b72a-2ea19411a9d6/fe7ca88c-2b6f-471d-ace9-d3d6a951e95f"
 					(reference "JP9")
@@
 		(dnp no)
 		(fields_autoplaced yes)
-		(property "Reference" "CP7"
+		(property "Reference" "CP5"
 			(at 142.24 113.0299 90)
 			(show_name no)
@@
 		(instances
 			(project "gateway2"
-				(path "/1800ee7d-fb6b-47f6-b72a-2ea19411a9d6/2270f938-9e88-4822-9195-66f8ec9fd89f"
-					(reference "CP7")
-					(unit 1)
-				)
-				(path "/1800ee7d-fb6b-47f6-b72a-2ea19411a9d6/48086788-2dae-4fa8-b688-a98b4725ecdb"
-					(reference "CP6")
-					(unit 1)
-				)
 				(path "/1800ee7d-fb6b-47f6-b72a-2ea19411a9d6/fe7ca88c-2b6f-471d-ace9-d3d6a951e95f"
 					(reference "CP5")
@@
 		(dnp no)
 		(fields_autoplaced yes)
-		(property "Reference" "#PWR077"
+		(property "Reference" "#PWR075"
 			(at 113.03 132.08 0)
 			(hide yes)
@@
 		(instances
 			(project "gateway2"
-				(path "/1800ee7d-fb6b-47f6-b72a-2ea19411a9d6/2270f938-9e88-4822-9195-66f8ec9fd89f"
-					(reference "#PWR077")
-					(unit 1)
-				)
-				(path "/1800ee7d-fb6b-47f6-b72a-2ea19411a9d6/48086788-2dae-4fa8-b688-a98b4725ecdb"
-					(reference "#PWR076")
-					(unit 1)
-				)
 				(path "/1800ee7d-fb6b-47f6-b72a-2ea19411a9d6/fe7ca88c-2b6f-471d-ace9-d3d6a951e95f"
 					(reference "#PWR075")
@@
 		(dnp yes)
 		(fields_autoplaced yes)
-		(property "Reference" "R40"
+		(property "Reference" "R35"
 			(at 173.99 82.5499 0)
 			(show_name no)
@@
 		(instances
 			(project "gateway2"
-				(path "/1800ee7d-fb6b-47f6-b72a-2ea19411a9d6/2270f938-9e88-4822-9195-66f8ec9fd89f"
-					(reference "R40")
-					(unit 1)
-				)
-				(path "/1800ee7d-fb6b-47f6-b72a-2ea19411a9d6/48086788-2dae-4fa8-b688-a98b4725ecdb"
-					(reference "R37")
-					(unit 1)
-				)
 				(path "/1800ee7d-fb6b-47f6-b72a-2ea19411a9d6/fe7ca88c-2b6f-471d-ace9-d3d6a951e95f"
 					(reference "R35")
@@
 		(dnp no)
 		(fields_autoplaced yes)
-		(property "Reference" "#PWR071"
+		(property "Reference" "#PWR069"
 			(at 181.61 132.08 0)
 			(hide yes)
@@
 		(instances
 			(project "gateway2"
-				(path "/1800ee7d-fb6b-47f6-b72a-2ea19411a9d6/2270f938-9e88-4822-9195-66f8ec9fd89f"
-					(reference "#PWR071")
-					(unit 1)
-				)
-				(path "/1800ee7d-fb6b-47f6-b72a-2ea19411a9d6/48086788-2dae-4fa8-b688-a98b4725ecdb"
-					(reference "#PWR070")
-					(unit 1)
-				)
 				(path "/1800ee7d-fb6b-47f6-b72a-2ea19411a9d6/fe7ca88c-2b6f-471d-ace9-d3d6a951e95f"
 					(reference "#PWR069")
@@
 		(dnp no)
 		(fields_autoplaced yes)
-		(property "Reference" "#PWR078"
+		(property "Reference" "#PWR079"
 			(at 104.14 119.38 0)
 			(hide yes)
@@
 		(instances
 			(project "gateway2"
-				(path "/1800ee7d-fb6b-47f6-b72a-2ea19411a9d6/2270f938-9e88-4822-9195-66f8ec9fd89f"
-					(reference "#PWR078")
-					(unit 1)
-				)
-				(path "/1800ee7d-fb6b-47f6-b72a-2ea19411a9d6/48086788-2dae-4fa8-b688-a98b4725ecdb"
-					(reference "#PWR080")
-					(unit 1)
-				)
 				(path "/1800ee7d-fb6b-47f6-b72a-2ea19411a9d6/fe7ca88c-2b6f-471d-ace9-d3d6a951e95f"
 					(reference "#PWR079")
@@
 		(in_pos_files yes)
 		(dnp no)
-		(property "Reference" "J10"
+		(property "Reference" "J8"
 			(at 101.6 96.5199 0)
 			(show_name no)
@@
 		(instances
 			(project "gateway2"
-				(path "/1800ee7d-fb6b-47f6-b72a-2ea19411a9d6/2270f938-9e88-4822-9195-66f8ec9fd89f"
-					(reference "J10")
-					(unit 1)
-				)
-				(path "/1800ee7d-fb6b-47f6-b72a-2ea19411a9d6/48086788-2dae-4fa8-b688-a98b4725ecdb"
-					(reference "J9")
-					(unit 1)
-				)
 				(path "/1800ee7d-fb6b-47f6-b72a-2ea19411a9d6/fe7ca88c-2b6f-471d-ace9-d3d6a951e95f"
 					(reference "J8")
@@
 		(in_pos_files yes)
 		(dnp no)
-		(property "Reference" "RN7"
+		(property "Reference" "RN5"
 			(at 149.86 107.696 90)
 			(show_name no)
@@
 		(instances
 			(project "gateway2"
-				(path "/1800ee7d-fb6b-47f6-b72a-2ea19411a9d6/2270f938-9e88-4822-9195-66f8ec9fd89f"
-					(reference "RN7")
-					(unit 1)
-				)
-				(path "/1800ee7d-fb6b-47f6-b72a-2ea19411a9d6/48086788-2dae-4fa8-b688-a98b4725ecdb"
-					(reference "RN6")
-					(unit 1)
-				)
 				(path "/1800ee7d-fb6b-47f6-b72a-2ea19411a9d6/fe7ca88c-2b6f-471d-ace9-d3d6a951e95f"
 					(reference "RN5")
@@
 		(dnp no)
 		(fields_autoplaced yes)
-		(property "Reference" "#PWR065"
+		(property "Reference" "#PWR063"
 			(at 137.16 132.08 0)
 			(hide yes)
@@
 		(instances
 			(project "gateway2"
-				(path "/1800ee7d-fb6b-47f6-b72a-2ea19411a9d6/2270f938-9e88-4822-9195-66f8ec9fd89f"
-					(reference "#PWR065")
-					(unit 1)
-				)
-				(path "/1800ee7d-fb6b-47f6-b72a-2ea19411a9d6/48086788-2dae-4fa8-b688-a98b4725ecdb"
-					(reference "#PWR064")
-					(unit 1)
-				)
 				(path "/1800ee7d-fb6b-47f6-b72a-2ea19411a9d6/fe7ca88c-2b6f-471d-ace9-d3d6a951e95f"
 					(reference "#PWR063")
@@
 		(in_pos_files yes)
 		(dnp no)
-		(property "Reference" "U10"
+		(property "Reference" "U8"
 			(at 188.722 92.964 0)
 			(show_name no)
@@
 		(instances
 			(project "gateway2"
-				(path "/1800ee7d-fb6b-47f6-b72a-2ea19411a9d6/2270f938-9e88-4822-9195-66f8ec9fd89f"
-					(reference "U10")
-					(unit 1)
-				)
-				(path "/1800ee7d-fb6b-47f6-b72a-2ea19411a9d6/48086788-2dae-4fa8-b688-a98b4725ecdb"
-					(reference "U9")
-					(unit 1)
-				)
 				(path "/1800ee7d-fb6b-47f6-b72a-2ea19411a9d6/fe7ca88c-2b6f-471d-ace9-d3d6a951e95f"
 					(reference "U8")
@@
 		(dnp no)
 		(fields_autoplaced yes)
-		(property "Reference" "JP14"
+		(property "Reference" "JP10"
 			(at 163.83 91.44 0)
 			(show_name no)
@@
 		(instances
 			(project "gateway2"
-				(path "/1800ee7d-fb6b-47f6-b72a-2ea19411a9d6/2270f938-9e88-4822-9195-66f8ec9fd89f"
-					(reference "JP14")
-					(unit 1)
-				)
-				(path "/1800ee7d-fb6b-47f6-b72a-2ea19411a9d6/48086788-2dae-4fa8-b688-a98b4725ecdb"
-					(reference "JP12")
-					(unit 1)
-				)
 				(path "/1800ee7d-fb6b-47f6-b72a-2ea19411a9d6/fe7ca88c-2b6f-471d-ace9-d3d6a951e95f"
 					(reference "JP10")
@@
 		(dnp no)
 		(fields_autoplaced yes)
-		(property "Reference" "#PWR083"
+		(property "Reference" "#PWR081"
 			(at 256.54 115.57 0)
 			(hide yes)
@@
 		(instances
 			(project "gateway2"
-				(path "/1800ee7d-fb6b-47f6-b72a-2ea19411a9d6/2270f938-9e88-4822-9195-66f8ec9fd89f"
-					(reference "#PWR083")
-					(unit 1)
-				)
-				(path "/1800ee7d-fb6b-47f6-b72a-2ea19411a9d6/48086788-2dae-4fa8-b688-a98b4725ecdb"
-					(reference "#PWR082")
-					(unit 1)
-				)
 				(path "/1800ee7d-fb6b-47f6-b72a-2ea19411a9d6/fe7ca88c-2b6f-471d-ace9-d3d6a951e95f"
 					(reference "#PWR081")
@@
 		(dnp no)
 		(fields_autoplaced yes)
-		(property "Reference" "C44"
+		(property "Reference" "C42"
 			(at 260.35 101.5999 0)
 			(show_name no)
@@
 		(instances
 			(project "gateway2"
-				(path "/1800ee7d-fb6b-47f6-b72a-2ea19411a9d6/2270f938-9e88-4822-9195-66f8ec9fd89f"
-					(reference "C44")
-					(unit 1)
-				)
-				(path "/1800ee7d-fb6b-47f6-b72a-2ea19411a9d6/48086788-2dae-4fa8-b688-a98b4725ecdb"
-					(reference "C43")
-					(unit 1)
-				)
 				(path "/1800ee7d-fb6b-47f6-b72a-2ea19411a9d6/fe7ca88c-2b6f-471d-ace9-d3d6a951e95f"
 					(reference "C42")

Commit message: Trying to fit 6 bricklet connectors.
Parts:
- renumbered C42 to C45, CP5 to CP6, J8 to J9, JP9 to JP11, JP10 to JP12, R34 to R36, R35 to R37, RN5 to RN6, U8 to U9

Commit message: Preparing for manufactoring.
Other:
- company: (none) -> ${COMPANY}
- title: (none) -> ${TITLE}
Changed lines of the file:
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@@
 	(generator_version "10.0")
 	(paper "A4")
+	(title_block
+		(title "${TITLE}")
+		(rev "${VERSION}")
+		(company "${COMPANY}")
+	)
 	(text "For some reason, Tinkerforge routes CS signal directly, \nskipping the buffer. Maybe it is related to their \nInfineon bug?.. Leaving it as an option."
 		(exclude_from_sim no)
