File: pcb/gateway/gateway2/Power.kicad_sch (KiCad schematic)
At the start: 14 parts, among them U3 RT6150AGQW

Commit message: Preparing for manufactoring.
Other:
- company: (none) -> ${COMPANY}
- title: (none) -> ${TITLE}
Changed lines of the file:
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@@
 	(generator_version "10.0")
 	(paper "A4")
+	(title_block
+		(title "${TITLE}")
+		(rev "${VERSION}")
+		(company "${COMPANY}")
+	)
 	(junction
 		(at 171.45 91.44)
